File: Flight computer/Hardware/circuit board design/GPS.sch (KiCad schematic (older format))
At the start: 0 parts

Commit message: Got the GPS wired up with the MAX-M8C.
I wired up the MCU to the GPS as well. Sensors are also wired up to the I2C line.

TODO:
-make everything run on 3.3V
- work out the pyro charges and drivers
many more.
Parts:
- added ANT1: Johanson1575, ICSSPicoTracker2:Johanson1575, symbol ICSSPicoTracker2-rescue:Johanson1575-ICSSPicoTracker
- added C67: 47pF, Capacitor_SMD:C_0402_1005Metric, symbol Device:C_Small
- added C68: 2.7pF, Capacitor_SMD:C_0402_1005Metric, symbol Device:C_Small
- added C72: 1nF, Capacitor_SMD:C_0402_1005Metric, symbol Device:C_Small
- added L20: 8.2nH, Inductor_SMD:L_0402_1005Metric, symbol Device:L_Small
- added L21: 6.8nH, Inductor_SMD:L_0402_1005Metric, symbol Device:L_Small
- added R2: 10K, symbol Device:R
- added R6: 47k, Resistor_SMD:R_0603_1608Metric, symbol Device:R_Small
- added U12: MAX2659ELT+, ICSSPicoTracker2:uDFN-6_1.0x1.5mm_P0.5mm, symbol ICSSPicoTracker2-rescue:MAX2659ELT+-ICSSPicoTracker
- added U13: SAFEB1G57KE0F00, ICSSPicoTracker2:Murata SAFE, symbol ICSSPicoTracker2-rescue:SAFEB1G57KE0F00-ICSSPicoTracker
- added U4: MAX-M8C, RF_GPS:ublox_MAX, symbol RF_GPS:MAX-M8C
Connections:
- net labels added: +3.3V, GND, GPS_1PPS, GPS_NRES, GPS_NSAFEBOOT, GPS_RXD, GPS_SCL, GPS_SDA, GPS_TXD
- wire segments 0 -> 49
Other:
- note added: "Arranged according to Figure 7 in the MAX-8 / MAX-M8 u-blox 8 / M8 GNSS modules Hardware Integration Manual. Page 12."
- note added: "Do we need the section that is already inside the MAX?\n"

Commit message: Connected the SPI connection with the SIlabs radio and the XTAL
Parts:
- removed R6: 47k, Resistor_SMD:R_0603_1608Metric, symbol Device:R_Small
Connections:
- wire segments 49 -> 46
Other:
- note added: "What are the capacitors and inductors for? they are not on the hardware integration manual\n"
Changed lines of the file:
@@
 	4900 2400 4900 2500
-$Comp
-L Device:R_Small R6
-U 1 1 5D5E3875
-P 5650 2150
-F 0 "R6" H 5709 2196 50  0000 L CNN
-F 1 "47k" H 5709 2105 50  0000 L CNN
-F 2 "Resistor_SMD:R_0603_1608Metric" H 5650 2150 50  0001 C CNN
-F 3 "~" H 5650 2150 50  0001 C CNN
-	1    5650 2150
-	1    0    0    -1
-$EndComp
-$Comp
-L power:GND #PWR074
-U 1 1 5D5E418A
-P 5650 2350
-F 0 "#PWR074" H 5650 2100 50  0001 C CNN
-F 1 "GND" H 5655 2177 50  0000 C CNN
-F 2 "" H 5650 2350 50  0001 C CNN
-F 3 "" H 5650 2350 50  0001 C CNN
-	1    5650 2350
-	1    0    0    -1
-$EndComp
-Wire Wire Line
-	5650 2350 5650 2250
 $Comp
 L Device:L_Small L21
@@
 Wire Wire Line
 	3000 2050 3250 2050
-Wire Wire Line
-	5650 2050 5650 1900
 $Comp
 L ICSSPicoTracker2-rescue:Johanson1575-ICSSPicoTracker ANT1
@@
 	1900 1500 1800 1500
 Wire Wire Line
-	5650 1900 6800 1900
-Wire Wire Line
 	5450 3650 4200 3650
 $Comp
@@
 	1    0    0    -1
 $EndComp
-Connection ~ 5650 1900
-Wire Wire Line
-	3250 1900 5650 1900
 Wire Wire Line
 	3250 2050 3250 1900
@@
 $EndComp
 $Bitmap
-Pos 9650 3400
-Scale 1.000000
+Pos 9200 2900
+Scale 2.000000
 Data
 89 50 4E 47 0D 0A 1A 0A 00 00 00 0D 49 48 44 52 00 00 02 CC 00 00 01 56 08 02 00 00 00 F2 A6 5C
@@
 EndData
 $EndBitmap
-Text Notes 8600 4150 0    50   ~ 0
+Text Notes 8500 4000 0    50   ~ 0
 Do we need the section that is already inside the MAX?\n
+Wire Wire Line
+	3250 1900 6800 1900
+Wire Notes Line
+	4200 1950 4200 2650
+Wire Notes Line
+	4200 2650 5250 2650
+Wire Notes Line
+	5250 2650 5250 1950
+Wire Notes Line
+	5250 1950 4200 1950
+Wire Notes Line
+	5000 1950 5000 1300
+Wire Notes Line
+	5000 1300 5300 1300
+Text Notes 4800 1250 0    50   ~ 0
+What are the capacitors and inductors for? they are not on the hardware integration manual\n
 $EndSCHEMATC

Commit message: changed boost converter resistor values for 3.3V and more
-started the pyro drivers
- connected the SPI connection between radio and MCU
- boost converter values changed.
Parts:
- ANT1: symbol ICSSPicoTracker2-rescue:Johanson1575-ICSSPicoTracker -> circuit-board-design-rescue:Johanson1575-ICSSPicoTracker-ICSSPicoTracker2-rescue
- U12: symbol ICSSPicoTracker2-rescue:MAX2659ELT+-ICSSPicoTracker -> circuit-board-design-rescue:MAX2659ELT+-ICSSPicoTracker-ICSSPicoTracker2-rescue
- U13: symbol ICSSPicoTracker2-rescue:SAFEB1G57KE0F00-ICSSPicoTracker -> circuit-board-design-rescue:SAFEB1G57KE0F00-ICSSPicoTracker-ICSSPicoTracker2-rescue
Connections:
- no-connect marks 0 -> 1
Other:
- note added: "http://www.explorelabs.com/blog/designing-a-gps-receiver/#ref-ublox-datasheet\n\nImportant info on why we use the components\n"
Changed lines of the file:
@@
 $Descr A4 11693 8268
 encoding utf-8
-Sheet 5 6
+Sheet 5 7
 Title ""
 Date ""
@@
 $EndDescr
 $Comp
-L ICSSPicoTracker2-rescue:MAX2659ELT+-ICSSPicoTracker U12
+L circuit-board-design-rescue:MAX2659ELT+-ICSSPicoTracker-ICSSPicoTracker2-rescue U12
 U 1 1 5D44B218
 P 2300 2350
@@
 $EndComp
 $Comp
-L ICSSPicoTracker2-rescue:SAFEB1G57KE0F00-ICSSPicoTracker U13
+L circuit-board-design-rescue:SAFEB1G57KE0F00-ICSSPicoTracker-ICSSPicoTracker2-rescue U13
 U 1 1 5D44BB5C
 P 3400 2450
@@
 	1    0    0    -1
 $EndComp
-$Comp
-L Device:C_Small C67
-U 1 1 5D45CE50
-P 4400 2200
-F 0 "C67" V 4171 2200 50  0000 C CNN
-F 1 "47pF" V 4262 2200 50  0000 C CNN
-F 2 "Capacitor_SMD:C_0402_1005Metric" H 4400 2200 50  0001 C CNN
-F 3 "~" H 4400 2200 50  0001 C CNN
-	1    4400 2200
-	0    1    1    0
-$EndComp
-$Comp
-L Device:L_Small L20
-U 1 1 5D45D95F
-P 4600 2450
-F 0 "L20" H 4450 2500 50  0000 L CNN
-F 1 "8.2nH" H 4350 2400 50  0000 L CNN
-F 2 "Inductor_SMD:L_0402_1005Metric" H 4600 2450 50  0001 C CNN
-F 3 "~" H 4600 2450 50  0001 C CNN
-	1    4600 2450
-	1    0    0    -1
-$EndComp
-$Comp
-L Device:C_Small C68
-U 1 1 5D45EA6D
-P 4900 2300
-F 0 "C68" H 4808 2254 50  0000 R CNN
-F 1 "2.7pF" H 4808 2345 50  0000 R CNN
-F 2 "Capacitor_SMD:C_0402_1005Metric" H 4900 2300 50  0001 C CNN
-F 3 "~" H 4900 2300 50  0001 C CNN
-	1    4900 2300
-	-1   0    0    1
-$EndComp
-Wire Wire Line
-	4600 2900 4600 2550
-Wire Wire Line
-	4600 2350 4600 2200
-Wire Wire Line
-	4600 2200 4500 2200
-Wire Wire Line
-	4900 2200 4600 2200
-Connection ~ 4600 2200
 Wire Wire Line
 	4150 2400 4250 2400
 Wire Wire Line
 	4250 2400 4250 2750
-Wire Wire Line
-	4150 2200 4300 2200
 Wire Wire Line
 	3300 2200 3000 2200
@@
 Wire Wire Line
 	2100 2200 2100 2550
-$Comp
-L power:GND #PWR061
-U 1 1 5D46AB52
-P 4900 2500
-F 0 "#PWR061" H 4900 2250 50  0001 C CNN
-F 1 "GND" H 4905 2327 50  0000 C CNN
-F 2 "" H 4900 2500 50  0001 C CNN
-F 3 "" H 4900 2500 50  0001 C CNN
-	1    4900 2500
-	1    0    0    -1
-$EndComp
-Wire Wire Line
-	4900 2400 4900 2500
 $Comp
 L Device:L_Small L21
@@
 	3000 2050 3250 2050
 $Comp
-L ICSSPicoTracker2-rescue:Johanson1575-ICSSPicoTracker ANT1
+L circuit-board-design-rescue:Johanson1575-ICSSPicoTracker-ICSSPicoTracker2-rescue ANT1
 U 1 1 5D521711
 P 1400 1500
@@
 Text Notes 4800 1250 0    50   ~ 0
 What are the capacitors and inductors for? they are not on the hardware integration manual\n
+Wire Wire Line
+	4900 2400 4900 2500
+$Comp
+L power:GND #PWR061
+U 1 1 5D46AB52
+P 4900 2500
+F 0 "#PWR061" H 4900 2250 50  0001 C CNN
+F 1 "GND" H 4905 2327 50  0000 C CNN
+F 2 "" H 4900 2500 50  0001 C CNN
+F 3 "" H 4900 2500 50  0001 C CNN
+	1    4900 2500
+	1    0    0    -1
+$EndComp
+Wire Wire Line
+	4150 2200 4300 2200
+Wire Wire Line
+	4900 2200 4600 2200
+Wire Wire Line
+	4600 2200 4500 2200
+Connection ~ 4600 2200
+Wire Wire Line
+	4600 2350 4600 2200
+Wire Wire Line
+	4600 2900 4600 2550
+$Comp
+L Device:C_Small C68
+U 1 1 5D45EA6D
+P 4900 2300
+F 0 "C68" H 4808 2254 50  0000 R CNN
+F 1 "2.7pF" H 4808 2345 50  0000 R CNN
+F 2 "Capacitor_SMD:C_0402_1005Metric" H 4900 2300 50  0001 C CNN
+F 3 "~" H 4900 2300 50  0001 C CNN
+	1    4900 2300
+	-1   0    0    1
+$EndComp
+$Comp
+L Device:L_Small L20
+U 1 1 5D45D95F
+P 4600 2450
+F 0 "L20" H 4450 2500 50  0000 L CNN
+F 1 "8.2nH" H 4350 2400 50  0000 L CNN
+F 2 "Inductor_SMD:L_0402_1005Metric" H 4600 2450 50  0001 C CNN
+F 3 "~" H 4600 2450 50  0001 C CNN
+	1    4600 2450
+	1    0    0    -1
+$EndComp
+$Comp
+L Device:C_Small C67
+U 1 1 5D45CE50
+P 4400 2200
+F 0 "C67" V 4171 2200 50  0000 C CNN
+F 1 "47pF" V 4262 2200 50  0000 C CNN
+F 2 "Capacitor_SMD:C_0402_1005Metric" H 4400 2200 50  0001 C CNN
+F 3 "~" H 4400 2200 50  0001 C CNN
+	1    4400 2200
+	0    1    1    0
+$EndComp
+Text Notes 7850 4950 0    50   ~ 0
+http://www.explorelabs.com/blog/designing-a-gps-receiver/#ref-ublox-datasheet\n\nImportant info on why we use the components\n
+NoConn ~ 5450 4250
 $EndSCHEMATC

Commit message: Wired up the SI4463 according to AN628 figure 16. Component values have not been set. Only type of component.
Parts:
- removed C67: 47pF, Capacitor_SMD:C_0402_1005Metric, symbol Device:C_Small
- removed C68: 2.7pF, Capacitor_SMD:C_0402_1005Metric, symbol Device:C_Small
- removed L20: 8.2nH, Inductor_SMD:L_0402_1005Metric, symbol Device:L_Small
Connections:
- wire segments 46 -> 42
Other:
- note removed: "What are the capacitors and inductors for? they are not on the hardware integration manual\n"
Changed lines of the file:
@@
 	1    0    0    -1
 $EndComp
-Wire Wire Line
-	5450 3950 4200 3950
 $Comp
 L power:GND #PWR052
@@
 	1    0    0    -1
 $EndComp
-Text HLabel 4200 3750 0    50   Output ~ 0
-GPS_TXD
-Text HLabel 4200 3650 0    50   Input ~ 0
-GPS_RXD
-Text HLabel 4200 4050 0    50   BiDi ~ 0
-GPS_SCL
-Text HLabel 4200 3950 0    50   BiDi ~ 0
-GPS_SDA
-Text HLabel 4200 4350 0    50   Input ~ 0
-GPS_NSAFEBOOT
-Text HLabel 4200 4450 0    50   Input ~ 0
-GPS_NRES
 Wire Wire Line
 	3000 2050 3250 2050
@@
 	1900 1500 1800 1500
 Wire Wire Line
-	5450 3650 4200 3650
-$Comp
-L power:GND #PWR011
-U 1 1 5D67FE0F
-P 6050 4900
-F 0 "#PWR011" H 6050 4650 50  0001 C CNN
-F 1 "GND" H 6055 4727 50  0000 C CNN
-F 2 "" H 6050 4900 50  0001 C CNN
-F 3 "" H 6050 4900 50  0001 C CNN
-	1    6050 4900
-	1    0    0    -1
-$EndComp
-Wire Wire Line
-	6800 3850 6650 3850
-Wire Wire Line
-	6800 1900 6800 3850
-Wire Wire Line
 	4600 2900 6900 2900
-$Comp
-L power:+3.3V #PWR010
-U 1 1 5D692740
-P 5850 3350
-F 0 "#PWR010" H 5850 3200 50  0001 C CNN
-F 1 "+3.3V" H 5865 3523 50  0000 C CNN
-F 2 "" H 5850 3350 50  0001 C CNN
-F 3 "" H 5850 3350 50  0001 C CNN
-	1    5850 3350
-	1    0    0    -1
-$EndComp
 Wire Wire Line
 	3250 2050 3250 1900
 Wire Wire Line
-	6250 3350 6250 1800
-Wire Wire Line
 	6250 1800 3150 1800
 Wire Wire Line
@@
 Wire Wire Line
 	3150 1900 3000 1900
-Wire Wire Line
-	6900 4050 6900 2900
-Wire Wire Line
-	6900 4050 6650 4050
 Text HLabel 7200 4350 2    50   Output ~ 0
 GPS_1PPS
-Wire Wire Line
-	6650 4350 7200 4350
 Text Notes 3000 5800 0    50   ~ 0
 Arranged according to Figure 7 in the MAX-8 / MAX-M8 u-blox 8 / M8 GNSS modules Hardware Integration Manual. Page 12.
-Wire Wire Line
-	6050 4900 6050 4800
-Wire Wire Line
-	6800 3850 6800 4800
-Wire Wire Line
-	6800 4800 6600 4800
-Connection ~ 6800 3850
-Connection ~ 6050 4800
-Wire Wire Line
-	6050 4800 6050 4750
-$Comp
-L Device:R R2
-U 1 1 5D69D778
-P 6450 4800
-F 0 "R2" V 6700 4800 50  0000 C CNN
-F 1 "10K" V 6600 4800 50  0000 C CNN
-F 2 "" V 6380 4800 50  0001 C CNN
-F 3 "~" H 6450 4800 50  0001 C CNN
-	1    6450 4800
-	0    1    1    0
-$EndComp
-Wire Wire Line
-	6300 4800 6050 4800
-Wire Wire Line
-	5450 4350 4200 4350
-Wire Wire Line
-	4200 3750 5450 3750
-Wire Wire Line
-	4200 4450 5450 4450
-Wire Wire Line
-	4200 4050 5450 4050
-$Comp
-L RF_GPS:MAX-M8C U4
-U 1 1 5D610F77
-P 6050 4050
-F 0 "U4" H 6050 4900 50  0000 C CNN
-F 1 "MAX-M8C" H 6050 5000 50  0000 C CNN
-F 2 "RF_GPS:ublox_MAX" H 6450 3400 50  0001 C CNN
-F 3 "https://www.u-blox.com/sites/default/files/MAX-M8-FW3_DataSheet_%28UBX-15031506%29.pdf" H 6050 4050 50  0001 C CNN
-	1    6050 4050
-	1    0    0    -1
-$EndComp
+Text Notes 8500 4000 0    50   ~ 0
+Do we need the section that is already inside the MAX?\n
+Wire Wire Line
+	3250 1900 6800 1900
+Text Notes 7850 4950 0    50   ~ 0
+http://www.explorelabs.com/blog/designing-a-gps-receiver/#ref-ublox-datasheet\n\nImportant info on why we use the components\n
+Wire Wire Line
+	4600 2200 4600 2900
+Wire Wire Line
+	4150 2200 4600 2200
+NoConn ~ 5450 4250
 $Bitmap
 Pos 9200 2900
@@
 EndData
 $EndBitmap
-Text Notes 8500 4000 0    50   ~ 0
-Do we need the section that is already inside the MAX?\n
-Wire Wire Line
-	3250 1900 6800 1900
-Wire Notes Line
-	4200 1950 4200 2650
-Wire Notes Line
-	4200 2650 5250 2650
-Wire Notes Line
-	5250 2650 5250 1950
-Wire Notes Line
-	5250 1950 4200 1950
-Wire Notes Line
-	5000 1950 5000 1300
-Wire Notes Line
-	5000 1300 5300 1300
-Text Notes 4800 1250 0    50   ~ 0
-What are the capacitors and inductors for? they are not on the hardware integration manual\n
-Wire Wire Line
-	4900 2400 4900 2500
 $Comp
-L power:GND #PWR061
-U 1 1 5D46AB52
-P 4900 2500
-F 0 "#PWR061" H 4900 2250 50  0001 C CNN
-F 1 "GND" H 4905 2327 50  0000 C CNN
-F 2 "" H 4900 2500 50  0001 C CNN
-F 3 "" H 4900 2500 50  0001 C CNN
-	1    4900 2500
+L RF_GPS:MAX-M8C U4
+U 1 1 5D610F77
+P 6050 4050
+F 0 "U4" H 6050 4900 50  0000 C CNN
+F 1 "MAX-M8C" H 6050 5000 50  0000 C CNN
+F 2 "RF_GPS:ublox_MAX" H 6450 3400 50  0001 C CNN
+F 3 "https://www.u-blox.com/sites/default/files/MAX-M8-FW3_DataSheet_%28UBX-15031506%29.pdf" H 6050 4050 50  0001 C CNN
+	1    6050 4050
 	1    0    0    -1
 $EndComp
 Wire Wire Line
-	4150 2200 4300 2200
-Wire Wire Line
-	4900 2200 4600 2200
-Wire Wire Line
-	4600 2200 4500 2200
-Connection ~ 4600 2200
-Wire Wire Line
-	4600 2350 4600 2200
-Wire Wire Line
-	4600 2900 4600 2550
+	4200 4050 5450 4050
+Wire Wire Line
+	4200 4450 5450 4450
+Wire Wire Line
+	4200 3750 5450 3750
+Wire Wire Line
+	5450 4350 4200 4350
+Wire Wire Line
+	6300 4800 6050 4800
 $Comp
-L Device:C_Small C68
-U 1 1 5D45EA6D
-P 4900 2300
-F 0 "C68" H 4808 2254 50  0000 R CNN
-F 1 "2.7pF" H 4808 2345 50  0000 R CNN
-F 2 "Capacitor_SMD:C_0402_1005Metric" H 4900 2300 50  0001 C CNN
-F 3 "~" H 4900 2300 50  0001 C CNN
-	1    4900 2300
-	-1   0    0    1
+L Device:R R2
+U 1 1 5D69D778
+P 6450 4800
+F 0 "R2" V 6700 4800 50  0000 C CNN
+F 1 "10K" V 6600 4800 50  0000 C CNN
+F 2 "" V 6380 4800 50  0001 C CNN
+F 3 "~" H 6450 4800 50  0001 C CNN
+	1    6450 4800
+	0    1    1    0
 $EndComp
+Wire Wire Line
+	6050 4800 6050 4750
+Connection ~ 6050 4800
+Connection ~ 6800 3850
+Wire Wire Line
+	6800 4800 6600 4800
+Wire Wire Line
+	6800 3850 6800 4800
+Wire Wire Line
+	6050 4900 6050 4800
+Wire Wire Line
+	6650 4350 7200 4350
+Wire Wire Line
+	6900 4050 6650 4050
+Wire Wire Line
+	6900 4050 6900 2900
+Wire Wire Line
+	6250 3350 6250 1800
 $Comp
-L Device:L_Small L20
-U 1 1 5D45D95F
-P 4600 2450
-F 0 "L20" H 4450 2500 50  0000 L CNN
-F 1 "8.2nH" H 4350 2400 50  0000 L CNN
-F 2 "Inductor_SMD:L_0402_1005Metric" H 4600 2450 50  0001 C CNN
-F 3 "~" H 4600 2450 50  0001 C CNN
-	1    4600 2450
+L power:+3.3V #PWR010
+U 1 1 5D692740
+P 5850 3350
+F 0 "#PWR010" H 5850 3200 50  0001 C CNN
+F 1 "+3.3V" H 5865 3523 50  0000 C CNN
+F 2 "" H 5850 3350 50  0001 C CNN
+F 3 "" H 5850 3350 50  0001 C CNN
+	1    5850 3350
 	1    0    0    -1
 $EndComp
+Wire Wire Line
+	6800 1900 6800 3850
+Wire Wire Line
+	6800 3850 6650 3850
 $Comp
-L Device:C_Small C67
-U 1 1 5D45CE50
-P 4400 2200
-F 0 "C67" V 4171 2200 50  0000 C CNN
-F 1 "47pF" V 4262 2200 50  0000 C CNN
-F 2 "Capacitor_SMD:C_0402_1005Metric" H 4400 2200 50  0001 C CNN
-F 3 "~" H 4400 2200 50  0001 C CNN
-	1    4400 2200
-	0    1    1    0
+L power:GND #PWR011
+U 1 1 5D67FE0F
+P 6050 4900
+F 0 "#PWR011" H 6050 4650 50  0001 C CNN
+F 1 "GND" H 6055 4727 50  0000 C CNN
+F 2 "" H 6050 4900 50  0001 C CNN
+F 3 "" H 6050 4900 50  0001 C CNN
+	1    6050 4900
+	1    0    0    -1
 $EndComp
-Text Notes 7850 4950 0    50   ~ 0
-http://www.explorelabs.com/blog/designing-a-gps-receiver/#ref-ublox-datasheet\n\nImportant info on why we use the components\n
-NoConn ~ 5450 4250
+Wire Wire Line
+	5450 3650 4200 3650
+Text HLabel 4200 4450 0    50   Input ~ 0
+GPS_NRES
+Text HLabel 4200 4350 0    50   Input ~ 0
+GPS_NSAFEBOOT
+Text HLabel 4200 3950 0    50   BiDi ~ 0
+GPS_SDA
+Text HLabel 4200 4050 0    50   BiDi ~ 0
+GPS_SCL
+Text HLabel 4200 3650 0    50   Input ~ 0
+GPS_RXD
+Text HLabel 4200 3750 0    50   Output ~ 0
+GPS_TXD
+Wire Wire Line
+	5450 3950 4200 3950
 $EndSCHEMATC

Commit message: changed all the paths for the schematic, footprints to local versions
so that it will not break when others access from another computer
Parts:
- ANT1: symbol circuit-board-design-rescue:Johanson1575-ICSSPicoTracker-ICSSPicoTracker2-rescue -> flight-computer:ICSSPicoTracker_Johanson1575
- U12: symbol circuit-board-design-rescue:MAX2659ELT+-ICSSPicoTracker-ICSSPicoTracker2-rescue -> flight-computer:ICSSPicoTracker_MAX2659ELT+
- U13: symbol circuit-board-design-rescue:SAFEB1G57KE0F00-ICSSPicoTracker-ICSSPicoTracker2-rescue -> flight-computer:ICSSPicoTracker_SAFEB1G57KE0F00
Connections:
- wire segments 42 -> 40
Other:
- note removed: "Do we need the section that is already inside the MAX?\n"
- moved on the sheet: C72, L21

Commit message: created net list for first time
-changed SAML21 to J variant7
-filled in foot prints for all components exept comparator
-changed the footprints of ICSS pico tracker to a local copy
Parts:
- ANT1: footprint ICSSPicoTracker2:Johanson1575 -> pico_tracker:Johanson1575
- R2: footprint (none) -> Resistor_SMD:R_0603_1608Metric
- U12: footprint ICSSPicoTracker2:uDFN-6_1.0x1.5mm_P0.5mm -> pico_tracker:uDFN-6_1.0x1.5mm_P0.5mm
- U13: footprint ICSSPicoTracker2:Murata SAFE -> pico_tracker:Murata SAFE
Changed lines of the file:
@@
 F 0 "U13" H 3725 2925 50  0000 C CNN
 F 1 "SAFEB1G57KE0F00" H 3725 2834 50  0000 C CNN
-F 2 "ICSSPicoTracker2:Murata SAFE" H 3400 2450 50  0001 C CNN
+F 2 "pico_tracker:Murata SAFE" H 3400 2450 50  0001 C CNN
 F 3 "https://www.murata.com/en-eu/products/productdata/8797690593310/DS-SAFEB1G57KE0F00.pdf?1453347007000" H 3400 2450 50  0001 C CNN
 	1    3400 2450
@@
 F 0 "ANT1" H 1250 1765 50  0000 C CNN
 F 1 "Johanson1575" H 1250 1674 50  0000 C CNN
-F 2 "ICSSPicoTracker2:Johanson1575" H 1300 1500 50  0001 C CNN
+F 2 "pico_tracker:Johanson1575" H 1300 1500 50  0001 C CNN
 F 3 "https://www.mouser.co.uk/datasheet/2/611/JTI_Antenna-1575AT43A40_2006-09-399627.pdf" H 1300 1500 50  0001 C CNN
 	1    1300 1500
@@
 F 0 "R2" V 6700 4800 50  0000 C CNN
 F 1 "10K" V 6600 4800 50  0000 C CNN
-F 2 "" V 6380 4800 50  0001 C CNN
+F 2 "Resistor_SMD:R_0603_1608Metric" V 6380 4800 50  0001 C CNN
 F 3 "~" H 6450 4800 50  0001 C CNN
 	1    6450 4800
@@
 F 0 "U12" H 2500 3115 50  0000 C CNN
 F 1 "MAX2659ELT+" H 2500 3024 50  0000 C CNN
-F 2 "ICSSPicoTracker2:uDFN-6_1.0x1.5mm_P0.5mm" H 2200 2350 50  0001 C CNN
+F 2 "pico_tracker:uDFN-6_1.0x1.5mm_P0.5mm" H 2200 2350 50  0001 C CNN
 F 3 "https://datasheets.maximintegrated.com/en/ds/MAX2659.pdf" H 2200 2350 50  0001 C CNN
 	1    2200 2350
