File: Flight computer/Hardware/circuit board design/GPS.sch (KiCad schematic (older format))
At the start: 7 parts, among them J6 Conn_Coaxial, U4 MAX-M8C

Commit message: added in the footprint for the 6 terminal block
routed the RF section with the 434 antenna
Parts:
- C12: value 2u2F -> 10uF
Changed lines of the file:
@@
 AR Path="/5D5B165E/5D99D56B" Ref="C12"  Part="1"
 F 0 "C12" H 5558 2896 50  0000 R CNN
-F 1 "2u2F" H 5558 2805 50  0000 R CNN
+F 1 "10uF" H 5558 2805 50  0000 R CNN
 F 2 "Capacitor_SMD:C_0603_1608Metric" H 5650 2850 50  0001 C CNN
 F 3 "~" H 5650 2850 50  0001 C CNN

Commit message: Finished routing the board with 3.3V power plane
Power for mosfets comes from 2mm tracks on top layer. Todo: make their connection to ground more robust
Connections:
- net +3V3: now also U4.6 (V_BCKP)
- no-connect marks 3 -> 2
Changed lines of the file:
@@
 Text Notes 7000 1150 0    50   ~ 0
 Layout according to MAX-8 / MAX-M8, \nHardware Integration Manual,\nSection 2.4.2 Antenna design with active antenna.
-NoConn ~ 6050 3350
 NoConn ~ 5450 4250
 Wire Wire Line
@@
 	6050 4750 6050 4900
 Wire Wire Line
-	5950 3350 5950 2650
+	5950 3350 5950 3300
 Wire Wire Line
 	5850 2650 5850 3350
@@
 Wire Wire Line
 	5300 3150 5300 3050
+Connection ~ 5300 3050
+Wire Wire Line
+	5300 3050 5650 3050
 $Comp
 L RF_GPS:MAX-M8C U4
@@
 	1    0    0    -1
 $EndComp
-Connection ~ 5300 3050
 Wire Wire Line
-	5300 3050 5650 3050
+	6050 3350 6050 3300
+Wire Wire Line
+	6050 3300 5950 3300
+Connection ~ 5950 3300
+Wire Wire Line
+	5950 3300 5950 2650
 $EndSCHEMATC

Commit message: updated links to purchasing several components
Parts:
- J6: Cost (none) -> 1.05; Purchase link (none) -> https://www.mouser.co.uk/ProductDetail/Hirose-Connector/UFL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
Changed lines of the file:
@@
 F 1 "Conn_Coaxial" H 8550 3934 50  0000 L CNN
 F 2 "Connector_Coaxial:U.FL_Hirose_U.FL-R-SMT-1_Vertical" H 8450 4050 50  0001 C CNN
-F 3 " ~" H 8450 4050 50  0001 C CNN
+F 3 "https://www.mouser.co.uk/datasheet/2/185/U.FL_catalog-939761.pdf" H 8450 4050 50  0001 C CNN
+F 4 "1.05" H 8450 4050 50  0001 C CNN "Cost"
+F 5 "https://www.mouser.co.uk/ProductDetail/Hirose-Connector/UFL-R-SMT01?qs=Ux3WWAnHpjDV3tCCbDi65g==" H 8450 4050 50  0001 C CNN "Purchase link"
 	1    8450 4050
 	1    0    0    -1
