File: Flight computer/Hardware/circuit board design/telemetry_radio.sch (KiCad schematic (older format))
At the start: 30 parts, among them U2 AS179-92LF, U3 Si4463, X1 32MHz TCXO

Commit message: Radio Update
Parts:
- L5: value 30nH -> 22nH
Connections:
- wire segments 109 -> 111
Other:
- moved on the sheet: C20
Changed lines of the file:
@@
 P 6550 2900
 F 0 "L5" V 6369 2900 50  0000 C CNN
-F 1 "30nH" V 6460 2900 50  0000 C CNN
+F 1 "22nH" V 6460 2900 50  0000 C CNN
 F 2 "" H 6550 2900 50  0001 C CNN
 F 3 "~" H 6550 2900 50  0001 C CNN
@@
 L power:+3.3V #PWR032
 U 1 1 5D6B5C3D
-P 1350 2900
-F 0 "#PWR032" H 1350 2750 50  0001 C CNN
-F 1 "+3.3V" H 1365 3073 50  0000 C CNN
-F 2 "" H 1350 2900 50  0001 C CNN
-F 3 "" H 1350 2900 50  0001 C CNN
-	1    1350 2900
+P 1550 2900
+F 0 "#PWR032" H 1550 2750 50  0001 C CNN
+F 1 "+3.3V" H 1565 3073 50  0000 C CNN
+F 2 "" H 1550 2900 50  0001 C CNN
+F 3 "" H 1550 2900 50  0001 C CNN
+	1    1550 2900
 	1    0    0    -1
 $EndComp
-NoConn ~ 1050 3600
+NoConn ~ 1250 3600
 $Comp
 L power:GND #PWR033
 U 1 1 5D6BDDD0
-P 1350 4100
-F 0 "#PWR033" H 1350 3850 50  0001 C CNN
-F 1 "GND" H 1355 3927 50  0000 C CNN
-F 2 "" H 1350 4100 50  0001 C CNN
-F 3 "" H 1350 4100 50  0001 C CNN
-	1    1350 4100
+P 1550 4100
+F 0 "#PWR033" H 1550 3850 50  0001 C CNN
+F 1 "GND" H 1555 3927 50  0000 C CNN
+F 2 "" H 1550 4100 50  0001 C CNN
+F 3 "" H 1550 4100 50  0001 C CNN
+	1    1550 4100
 	1    0    0    -1
 $EndComp
 Wire Wire Line
-	3400 4450 1950 4450
+	3400 4450 2300 4450
 $Comp
 L Device:C_Small C20
 U 1 1 5D6C2DE3
-P 1950 3900
-F 0 "C20" H 2200 3900 50  0000 C CNN
-F 1 "10nF" H 2200 3800 50  0000 C CNN
-F 2 "" H 1950 3900 50  0001 C CNN
-F 3 "~" H 1950 3900 50  0001 C CNN
-	1    1950 3900
+P 2300 3900
+F 0 "C20" H 2550 3900 50  0000 C CNN
+F 1 "10nF" H 2550 3800 50  0000 C CNN
+F 2 "" H 2300 3900 50  0001 C CNN
+F 3 "~" H 2300 3900 50  0001 C CNN
+	1    2300 3900
 	1    0    0    1
 $EndComp
@@
 $EndComp
 Wire Wire Line
-	1350 2900 1350 3150
-Wire Wire Line
-	1350 3900 1350 4000
+	1550 2900 1550 3150
+Wire Wire Line
+	1550 3900 1550 4000
 $Comp
 L Oscillator:IQXO-70 X1
 U 1 1 5D766DA4
-P 1350 3600
-F 0 "X1" H 1694 3646 50  0000 L CNN
-F 1 "32MHz TCXO" H 1400 3350 50  0000 L CNN
-F 2 "Oscillator:Oscillator_SMD_IQD_IQXO70-4Pin_7.5x5.0mm" H 2025 3275 50  0001 C CNN
-F 3 "http://www.iqdfrequencyproducts.com/products/details/iqxo-70-11-30.pdf" H 1250 3600 50  0001 C CNN
-	1    1350 3600
+P 1550 3600
+F 0 "X1" H 1894 3646 50  0000 L CNN
+F 1 "32MHz TCXO" H 1600 3350 50  0000 L CNN
+F 2 "Oscillator:Oscillator_SMD_IQD_IQXO70-4Pin_7.5x5.0mm" H 2225 3275 50  0001 C CNN
+F 3 "http://www.iqdfrequencyproducts.com/products/details/iqxo-70-11-30.pdf" H 1450 3600 50  0001 C CNN
+	1    1550 3600
 	1    0    0    -1
 $EndComp
 Wire Wire Line
-	800  3150 1350 3150
-Connection ~ 1350 3150
-Wire Wire Line
-	1350 3150 1350 3300
+	800  3150 1550 3150
+Connection ~ 1550 3150
+Wire Wire Line
+	1550 3150 1550 3300
 Wire Wire Line
 	800  3600 800  4000
 Wire Wire Line
-	800  4000 1350 4000
-Connection ~ 1350 4000
-Wire Wire Line
-	1350 4000 1350 4100
-Wire Wire Line
-	1650 3600 1950 3600
-Wire Wire Line
-	1950 3600 1950 3800
-Wire Wire Line
-	1950 4000 1950 4450
+	800  4000 1550 4000
+Connection ~ 1550 4000
+Wire Wire Line
+	1550 4000 1550 4100
+Wire Wire Line
+	1850 3600 2300 3600
+Wire Wire Line
+	2300 3600 2300 3800
+Wire Wire Line
+	2300 4000 2300 4450
 Wire Wire Line
 	8100 3500 8100 3600
@@
 Wire Notes Line
 	6450 4200 5050 4200
+Wire Wire Line
+	4200 4250 4700 4250
+Wire Wire Line
+	4700 4250 4700 2900
+Connection ~ 4700 2900
 $EndSCHEMATC

Commit message: created net list for first time
-changed SAML21 to J variant7
-filled in foot prints for all components exept comparator
-changed the footprints of ICSS pico tracker to a local copy
Parts:
- AE1: footprint (none) -> pico_tracker:Yageo434; symbol Device:Antenna -> flight-computer:ICSSPicoTracker_Yageo434
- C10, C19, C22, C23: footprint (none) -> Capacitor_SMD:C_0603_1608Metric
- C11, C12, C13, C14, C15, C16, C17, C18, C20, C21, C24, C25, C26, C27, C8: footprint (none) -> Capacitor_SMD:C_0402_1005Metric
- L2, L3, L4, L5, L6, L7, L8: footprint (none) -> Inductor_SMD:L_0402_1005Metric
Connections:
- wire segments 111 -> 112
- no-connect marks 3 -> 4
Changed lines of the file:
@@
 F 0 "C18" V 5571 2900 50  0000 C CNN
 F 1 "9.1pF" V 5662 2900 50  0000 C CNN
-F 2 "" H 5800 2900 50  0001 C CNN
+F 2 "Capacitor_SMD:C_0402_1005Metric" H 5800 2900 50  0001 C CNN
 F 3 "~" H 5800 2900 50  0001 C CNN
 	1    5800 2900
@@
 F 0 "L5" V 6369 2900 50  0000 C CNN
 F 1 "22nH" V 6460 2900 50  0000 C CNN
-F 2 "" H 6550 2900 50  0001 C CNN
+F 2 "Inductor_SMD:L_0402_1005Metric" H 6550 2900 50  0001 C CNN
 F 3 "~" H 6550 2900 50  0001 C CNN
 	1    6550 2900
@@
 F 0 "L6" V 5750 4650 50  0000 C CNN
 F 1 "62nH" V 5650 4650 50  0000 C CNN
-F 2 "" H 5550 4650 50  0001 C CNN
+F 2 "Inductor_SMD:L_0402_1005Metric" H 5550 4650 50  0001 C CNN
 F 3 "~" H 5550 4650 50  0001 C CNN
 	1    5550 4650
@@
 F 0 "C17" H 5342 5004 50  0000 L CNN
 F 1 "4.7pF" H 5342 5095 50  0000 L CNN
-F 2 "" H 5250 5050 50  0001 C CNN
+F 2 "Capacitor_SMD:C_0402_1005Metric" H 5250 5050 50  0001 C CNN
 F 3 "~" H 5250 5050 50  0001 C CNN
 	1    5250 5050
@@
 F 0 "C14" H 6992 3296 50  0000 L CNN
 F 1 "12pF" H 6992 3205 50  0000 L CNN
-F 2 "" H 6900 3250 50  0001 C CNN
+F 2 "Capacitor_SMD:C_0402_1005Metric" H 6900 3250 50  0001 C CNN
 F 3 "~" H 6900 3250 50  0001 C CNN
 	1    6900 3250
@@
 F 0 "C16" H 6350 3300 50  0000 L CNN
 F 1 "15pF" H 6350 3200 50  0000 L CNN
-F 2 "" H 6200 3250 50  0001 C CNN
+F 2 "Capacitor_SMD:C_0402_1005Metric" H 6200 3250 50  0001 C CNN
 F 3 "~" H 6200 3250 50  0001 C CNN
 	1    6200 3250
@@
 F 0 "C13" V 7463 3100 50  0000 C CNN
 F 1 "150pF" V 7372 3100 50  0000 C CNN
-F 2 "" H 7600 3100 50  0001 C CNN
+F 2 "Capacitor_SMD:C_0402_1005Metric" H 7600 3100 50  0001 C CNN
 F 3 "~" H 7600 3100 50  0001 C CNN
 	1    7600 3100
@@
 F 0 "L3" V 7019 2900 50  0000 C CNN
 F 1 "18nH" V 7110 2900 50  0000 C CNN
-F 2 "" H 7200 2900 50  0001 C CNN
+F 2 "Inductor_SMD:L_0402_1005Metric" H 7200 2900 50  0001 C CNN
 F 3 "~" H 7200 2900 50  0001 C CNN
 	1    7200 2900
@@
 F 0 "C20" H 2550 3900 50  0000 C CNN
 F 1 "10nF" H 2550 3800 50  0000 C CNN
-F 2 "" H 2300 3900 50  0001 C CNN
+F 2 "Capacitor_SMD:C_0402_1005Metric" H 2300 3900 50  0001 C CNN
 F 3 "~" H 2300 3900 50  0001 C CNN
 	1    2300 3900
@@
 F 0 "C21" H 1050 3500 50  0000 C CNN
 F 1 "33nF" H 1050 3400 50  0000 C CNN
-F 2 "" H 800 3500 50  0001 C CNN
+F 2 "Capacitor_SMD:C_0402_1005Metric" H 800 3500 50  0001 C CNN
 F 3 "~" H 800 3500 50  0001 C CNN
 	1    800  3500
@@
 F 0 "C11" V 8571 3000 50  0000 C CNN
 F 1 "150pF" V 8662 3000 50  0000 C CNN
-F 2 "" H 8800 3000 50  0001 C CNN
+F 2 "Capacitor_SMD:C_0402_1005Metric" H 8800 3000 50  0001 C CNN
 F 3 "~" H 8800 3000 50  0001 C CNN
 	1    8800 3000
@@
 $EndComp
 $Comp
-L Device:Antenna AE1
+L flight-computer:ICSSPicoTracker_Yageo434 AE1
 U 1 1 5D6B791C
-P 10900 2400
-F 0 "AE1" H 10980 2389 50  0000 L CNN
-F 1 "Antenna" H 10980 2298 50  0000 L CNN
-F 2 "" H 10900 2400 50  0001 C CNN
-F 3 "~" H 10900 2400 50  0001 C CNN
-	1    10900 2400
-	-1   0    0    -1
-$EndComp
-Wire Wire Line
-	10900 3000 10900 2600
+P 10150 2250
+F 0 "AE1" H 10150 2650 50  0000 L CNN
+F 1 "Antenna" H 10100 2500 50  0000 L CNN
+F 2 "pico_tracker:Yageo434" H 10150 2250 50  0001 C CNN
+F 3 "~" H 10150 2250 50  0001 C CNN
+	1    10150 2250
+	-1   0    0    -1
+$EndComp
 Wire Notes Line
 	10400 3850 9000 3850
@@
 F 0 "L2" V 9569 3000 50  0000 C CNN
 F 1 "0R" V 9660 3000 50  0000 C CNN
-F 2 "" H 9750 3000 50  0001 C CNN
+F 2 "Inductor_SMD:L_0402_1005Metric" H 9750 3000 50  0001 C CNN
 F 3 "~" H 9750 3000 50  0001 C CNN
 	1    9750 3000
@@
 F 0 "C8" H 10142 3346 50  0000 L CNN
 F 1 "NF" H 10142 3255 50  0000 L CNN
-F 2 "" H 10050 3300 50  0001 C CNN
+F 2 "Capacitor_SMD:C_0402_1005Metric" H 10050 3300 50  0001 C CNN
 F 3 "~" H 10050 3300 50  0001 C CNN
 	1    10050 3300
@@
 F 0 "C26" H 9492 3346 50  0000 L CNN
 F 1 "NF" H 9492 3255 50  0000 L CNN
-F 2 "" H 9400 3300 50  0001 C CNN
+F 2 "Capacitor_SMD:C_0402_1005Metric" H 9400 3300 50  0001 C CNN
 F 3 "~" H 9400 3300 50  0001 C CNN
 	1    9400 3300
@@
 Connection ~ 9400 3000
 Wire Wire Line
-	10050 3000 10900 3000
+	10050 3000 10600 3000
 $Comp
 L RF_Switch:AS179-92LF U2
@@
 F 0 "C12" V 7371 2900 50  0000 C CNN
 F 1 "150pF" V 7462 2900 50  0000 C CNN
-F 2 "" H 7600 2900 50  0001 C CNN
+F 2 "Capacitor_SMD:C_0402_1005Metric" H 7600 2900 50  0001 C CNN
 F 3 "~" H 7600 2900 50  0001 C CNN
 	1    7600 2900
@@
 F 0 "C22" H 3908 3646 50  0000 R CNN
 F 1 "1uF" H 3908 3555 50  0000 R CNN
-F 2 "" H 4000 3600 50  0001 C CNN
+F 2 "Capacitor_SMD:C_0603_1608Metric" H 4000 3600 50  0001 C CNN
 F 3 "~" H 4000 3600 50  0001 C CNN
 	1    4000 3600
@@
 F 0 "C23" H 4258 3646 50  0000 R CNN
 F 1 "100nF" H 4258 3555 50  0000 R CNN
-F 2 "" H 4350 3600 50  0001 C CNN
+F 2 "Capacitor_SMD:C_0603_1608Metric" H 4350 3600 50  0001 C CNN
 F 3 "~" H 4350 3600 50  0001 C CNN
 	1    4350 3600
@@
 F 0 "C10" H 3208 2496 50  0000 R CNN
 F 1 "2.2uF" H 3208 2405 50  0000 R CNN
-F 2 "" H 3300 2450 50  0001 C CNN
+F 2 "Capacitor_SMD:C_0603_1608Metric" H 3300 2450 50  0001 C CNN
 F 3 "~" H 3300 2450 50  0001 C CNN
 	1    3300 2450
@@
 F 0 "C15" H 4008 2496 50  0000 R CNN
 F 1 "33pF" H 4008 2405 50  0000 R CNN
-F 2 "" H 4100 2450 50  0001 C CNN
+F 2 "Capacitor_SMD:C_0402_1005Metric" H 4100 2450 50  0001 C CNN
 F 3 "~" H 4100 2450 50  0001 C CNN
 	1    4100 2450
@@
 F 0 "L8" H 4656 2454 50  0000 R CNN
 F 1 "220nH" H 4656 2545 50  0000 R CNN
-F 2 "" H 4700 2500 50  0001 C CNN
+F 2 "Inductor_SMD:L_0402_1005Metric" H 4700 2500 50  0001 C CNN
 F 3 "~" H 4700 2500 50  0001 C CNN
 	1    4700 2500
@@
 F 0 "C19" H 3608 2496 50  0000 R CNN
 F 1 "100nf" H 3608 2405 50  0000 R CNN
-F 2 "" H 3700 2450 50  0001 C CNN
+F 2 "Capacitor_SMD:C_0603_1608Metric" H 3700 2450 50  0001 C CNN
 F 3 "~" H 3700 2450 50  0001 C CNN
 	1    3700 2450
@@
 F 0 "C24" H 8592 4446 50  0000 L CNN
 F 1 "1nF" H 8592 4355 50  0000 L CNN
-F 2 "" H 8500 4400 50  0001 C CNN
+F 2 "Capacitor_SMD:C_0402_1005Metric" H 8500 4400 50  0001 C CNN
 F 3 "~" H 8500 4400 50  0001 C CNN
 	1    8500 4400
@@
 F 0 "C25" H 9058 4446 50  0000 R CNN
 F 1 "1nF" H 9058 4355 50  0000 R CNN
-F 2 "" H 9150 4400 50  0001 C CNN
+F 2 "Capacitor_SMD:C_0402_1005Metric" H 9150 4400 50  0001 C CNN
 F 3 "~" H 9150 4400 50  0001 C CNN
 	1    9150 4400
@@
 F 0 "L4" V 5219 2900 50  0000 C CNN
 F 1 "30nH" V 5310 2900 50  0000 C CNN
-F 2 "" H 5400 2900 50  0001 C CNN
+F 2 "Inductor_SMD:L_0402_1005Metric" H 5400 2900 50  0001 C CNN
 F 3 "~" H 5400 2900 50  0001 C CNN
 	1    5400 2900
@@
 F 0 "L7" V 5962 4350 50  0000 C CNN
 F 1 "62nH" V 5871 4350 50  0000 C CNN
-F 2 "" H 6050 4350 50  0001 C CNN
+F 2 "Inductor_SMD:L_0402_1005Metric" H 6050 4350 50  0001 C CNN
 F 3 "~" H 6050 4350 50  0001 C CNN
 	1    6050 4350
@@
 F 0 "C27" V 5913 4850 50  0000 C CNN
 F 1 "4.7pF" V 5822 4850 50  0000 C CNN
-F 2 "" H 6050 4850 50  0001 C CNN
+F 2 "Capacitor_SMD:C_0402_1005Metric" H 6050 4850 50  0001 C CNN
 F 3 "~" H 6050 4850 50  0001 C CNN
 	1    6050 4850
@@
 	4700 4250 4700 2900
 Connection ~ 4700 2900
+Wire Wire Line
+	10550 2250 10600 2250
+Wire Wire Line
+	10600 2250 10600 3000
+NoConn ~ 9850 2250
 $EndSCHEMATC

Commit message: more upgrades
- removed the comparators
- added the cost and link to buy components
- added in a symbol for USB
Parts:
- removed X1: 32MHz TCXO, Oscillator:Oscillator_SMD_IQD_IQXO70-4Pin_7.5x5.0mm, symbol Oscillator:IQXO-70
- added X1: TM-32.000-AF3-33-S-Oscillator, Oscillator:Oscillator_SMD_SeikoEpson_SG210-4Pin_2.5x2.0mm_HandSoldering, symbol flight-computer:TM-32.000-AF3-33-S-Oscillator
- ANT2: renamed from AE1; value Antenna -> ICSSPicoTracker_Yageo434; Cost (none) -> 1.33; Purchase link (none) -> https://www.mouser.co.uk/ProductDetail/Yageo/ANT1204F002R04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
Changed lines of the file:
@@
 $EndComp
 $Comp
-L flight-computer:ICSSPicoTracker_Yageo434 AE1
+L flight-computer:ICSSPicoTracker_Yageo434 ANT2
 U 1 1 5D6B791C
 P 10150 2250
-F 0 "AE1" H 10150 2650 50  0000 L CNN
-F 1 "Antenna" H 10100 2500 50  0000 L CNN
+F 0 "ANT2" H 10150 2650 50  0000 L CNN
+F 1 "ICSSPicoTracker_Yageo434" H 10100 2500 50  0000 L CNN
 F 2 "pico_tracker:Yageo434" H 10150 2250 50  0001 C CNN
-F 3 "~" H 10150 2250 50  0001 C CNN
+F 3 "https://www.mouser.co.uk/datasheet/2/447/An_SMD_UHF_433_1204_0-595178.pdf" H 10150 2250 50  0001 C CNN
+F 4 "https://www.mouser.co.uk/ProductDetail/Yageo/ANT1204F002R0433A?qs=CqAAFKzD4h9Rz96OVrhbMw%3D%3D" H 10150 2250 50  0001 C CNN "Purchase link"
+F 5 "1.33" H 10150 2250 50  0001 C CNN "Cost"
 	1    10150 2250
 	-1   0    0    -1
@@
 Wire Wire Line
 	1550 3900 1550 4000
-$Comp
-L Oscillator:IQXO-70 X1
-U 1 1 5D766DA4
-P 1550 3600
-F 0 "X1" H 1894 3646 50  0000 L CNN
-F 1 "32MHz TCXO" H 1600 3350 50  0000 L CNN
-F 2 "Oscillator:Oscillator_SMD_IQD_IQXO70-4Pin_7.5x5.0mm" H 2225 3275 50  0001 C CNN
-F 3 "http://www.iqdfrequencyproducts.com/products/details/iqxo-70-11-30.pdf" H 1450 3600 50  0001 C CNN
-	1    1550 3600
-	1    0    0    -1
-$EndComp
 Wire Wire Line
 	800  3150 1550 3150
@@
 	10600 2250 10600 3000
 NoConn ~ 9850 2250
+$Comp
+L flight-computer:TM-32.000-AF3-33-S-Oscillator X1
+U 1 1 5D703E49
+P 1550 3600
+F 0 "X1" H 1500 4800 50  0000 L CNN
+F 1 "TM-32.000-AF3-33-S-Oscillator" H 1000 4700 50  0000 L CNN
+F 2 "Oscillator:Oscillator_SMD_SeikoEpson_SG210-4Pin_2.5x2.0mm_HandSoldering" H 2000 3250 50  0001 C CNN
+F 3 "https://docs-emea.rs-online.com/webdocs/15dc/0900766b815dc7d9.pdf" H 1450 3600 50  0001 C CNN
+F 4 "3.43" H 1550 3600 50  0001 C CNN "Cost"
+F 5 "https://uk.rs-online.com/web/p/tcxo-oscillators/1442366/" H 1550 3600 50  0001 C CNN "Purchase link"
+	1    1550 3600
+	1    0    0    -1
+$EndComp
 $EndSCHEMATC

Commit message: added in LDO based power supply
Parts:
- U2: Cost (none) -> 0.946; Purchase link (none) -> https://www.mouser.co.uk/ProductDetail/Skyworks-Solutions-I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
Changed lines of the file:
@@
 F 2 "Package_TO_SOT_SMD:SOT-363_SC-70-6" H 8300 3100 50  0001 C CNN
 F 3 "http://www.skyworksinc.com/uploads/documents/AS179_92LF_200176H.pdf" H 8300 3100 50  0001 C CNN
+F 4 "0.946" H 8200 3100 50  0001 C CNN "Cost"
+F 5 "https://www.mouser.co.uk/ProductDetail/Skyworks-Solutions-Inc/AS179-92LF?qs=sGAEpiMZZMsdcLTUVTS%2FgBfPoKwZ3liX" H 8200 3100 50  0001 C CNN "Purchase link"
 	1    8200 3100
 	-1   0    0    -1

Commit message: made some attempts to route the board
-replaced footprint for Radio TCXO
Parts:
- X1: footprint Oscillator:Oscillator_SMD_SeikoEpson_SG210-4Pin_2.5x2.0mm_HandSoldering -> Crystal:Crystal_SMD_2520-4Pin_2.5x2.0mm
Changed lines of the file:
@@
 F 0 "X1" H 1500 4800 50  0000 L CNN
 F 1 "TM-32.000-AF3-33-S-Oscillator" H 1000 4700 50  0000 L CNN
-F 2 "Oscillator:Oscillator_SMD_SeikoEpson_SG210-4Pin_2.5x2.0mm_HandSoldering" H 2000 3250 50  0001 C CNN
+F 2 "Crystal:Crystal_SMD_2520-4Pin_2.5x2.0mm" H 2000 3250 50  0001 C CNN
 F 3 "https://docs-emea.rs-online.com/webdocs/15dc/0900766b815dc7d9.pdf" H 1450 3600 50  0001 C CNN
 F 4 "3.43" H 1550 3600 50  0001 C CNN "Cost"

Commit message: changed the footprint for 220 nH inductor and removed the circuit for low power voltage measurments
Parts:
- L8: footprint Inductor_SMD:L_0402_1005Metric -> Inductor_SMD:L_0603_1608Metric
Changed lines of the file:
@@
 F 0 "L8" H 4656 2454 50  0000 R CNN
 F 1 "220nH" H 4656 2545 50  0000 R CNN
-F 2 "Inductor_SMD:L_0402_1005Metric" H 4700 2500 50  0001 C CNN
+F 2 "Inductor_SMD:L_0603_1608Metric" H 4700 2500 50  0001 C CNN
 F 3 "~" H 4700 2500 50  0001 C CNN
 	1    4700 2500

Commit message: moved gps antenna coax connection to right page
Parts:
- added U?: 0433BM41A0019E, Johanson_frontend:BALUN_0433BM41A0019E, symbol 0433BM41A0019E:0433BM41A0019E
Changed lines of the file:
@@
+	1    0    0    -1
+$EndComp
+$Comp
+L 0433BM41A0019E:0433BM41A0019E U?
+U 1 1 5D767292
+P 6550 1350
+F 0 "U?" H 6550 1867 50  0000 C CNN
+F 1 "0433BM41A0019E" H 6550 1776 50  0000 C CNN
+F 2 "Johanson_frontend:BALUN_0433BM41A0019E" H 6050 2000 50  0001 L BNN
+F 3 "https://www.johansontechnology.com/datasheets/0433BM41A0019/0433BM41A0019.pdf" H 6050 2000 50  0001 L BNN
+	1    6550 1350
 	1    0    0    -1
 $EndComp
