File: Flight computer/Hardware/circuit board design/_autosave-circuit board design.kicad_pcb (KiCad board)
At the start: 4 copper layers, 30.5 x 82.6 mm, 90 parts, among them J1 Conn_01x05, J2 USB_B_Micro, J3 Screw_Terminal_01x04, J4 Conn_01x02, J5 Screw_Terminal_01x04, J6 Conn_Coaxial, J7 Conn_Coaxial, U1 IIS2MDC, U10 BMI088, U11 ATSAML21J18B-AUT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

Commit message: tried routing first round
Parts:
- moved U5 54.3 mm to (254.4, 262.4)
- moved R12 5.48 mm to (276.7, 275.8)
- moved C89 2.56 mm to (276.7, 274.3), turned to 180 degrees
- moved R13 0.76 mm to (274.4, 275.1)
- moved R3 0.76 mm to (272.9, 275.1)
Routing:
- net GND: track 141.1 -> 152.1 mm, vias 37 -> 41
- net +3V3: track 69.6 -> 74.8 mm
- net Net-(C89-Pad1): track 0.00 -> 4.04 mm
