File: Flight computer/Hardware/circuit board design/pyro_driver.sch (KiCad schematic (older format))
At the start: 17 parts, among them J3 Screw_Terminal_01x04, J5 Screw_Terminal_01x04, SW1 SW_DPST, U5 Si7232DN, U6 Si7232DN

Commit message: updated the datasheet links and sites to purchase
Parts:
- J3, J5: Cost (none) -> 0.71; Purchase link (none) -> https://uk.rs-online.com/web/p/pcb-terminal-blocks/3617689/
Changed lines of the file:
@@
 F 1 "Screw_Terminal_01x04" H 8418 3066 50  0000 C CNN
 F 2 "TerminalBlock_TE-Connectivity:TerminalBlock_TE_282834-4_1x04_P2.54mm_Horizontal" H 8500 3400 50  0001 C CNN
-F 3 "~" H 8500 3400 50  0001 C CNN
+F 3 "https://docs-emea.rs-online.com/webdocs/002d/0900766b8002dc8a.pdf" H 8500 3400 50  0001 C CNN
+F 4 "0.71" H 8500 3400 50  0001 C CNN "Cost"
+F 5 "https://uk.rs-online.com/web/p/pcb-terminal-blocks/3617689/" H 8500 3400 50  0001 C CNN "Purchase link"
 	1    8500 3400
 	-1   0    0    1
@@
 F 1 "Screw_Terminal_01x04" H 8418 4116 50  0000 C CNN
 F 2 "TerminalBlock_TE-Connectivity:TerminalBlock_TE_282834-4_1x04_P2.54mm_Horizontal" H 8500 4450 50  0001 C CNN
-F 3 "~" H 8500 4450 50  0001 C CNN
+F 3 "https://docs-emea.rs-online.com/webdocs/002d/0900766b8002dc8a.pdf" H 8500 4450 50  0001 C CNN
+F 4 "0.71" H 8500 4450 50  0001 C CNN "Cost"
+F 5 "https://uk.rs-online.com/web/p/pcb-terminal-blocks/3617689/" H 8500 4450 50  0001 C CNN "Purchase link"
 	1    8500 4450
 	-1   0    0    1

Commit message: swapped out the 434 wire antenna for a Yageo434 chip antenna for smaller form factor
I put in the 3D model for the te connectivity terminal blocks
Parts:
- J3, J5: footprint TerminalBlock_TE-Connectivity:TerminalBlock_TE_282834-4_1x04_P2.54mm_Horizontal -> flight-computer:TerminalBlock_TE_282834-4_1x04_P2.54mm_Horizontal
Changed lines of the file:
@@
 F 0 "J3" H 8418 2975 50  0000 C CNN
 F 1 "Screw_Terminal_01x04" H 8418 3066 50  0000 C CNN
-F 2 "TerminalBlock_TE-Connectivity:TerminalBlock_TE_282834-4_1x04_P2.54mm_Horizontal" H 8500 3400 50  0001 C CNN
+F 2 "flight-computer:TerminalBlock_TE_282834-4_1x04_P2.54mm_Horizontal" H 8500 3400 50  0001 C CNN
 F 3 "https://docs-emea.rs-online.com/webdocs/002d/0900766b8002dc8a.pdf" H 8500 3400 50  0001 C CNN
 F 4 "0.71" H 8500 3400 50  0001 C CNN "Cost"
@@
 F 0 "J5" H 8418 4025 50  0000 C CNN
 F 1 "Screw_Terminal_01x04" H 8418 4116 50  0000 C CNN
-F 2 "TerminalBlock_TE-Connectivity:TerminalBlock_TE_282834-4_1x04_P2.54mm_Horizontal" H 8500 4450 50  0001 C CNN
+F 2 "flight-computer:TerminalBlock_TE_282834-4_1x04_P2.54mm_Horizontal" H 8500 4450 50  0001 C CNN
 F 3 "https://docs-emea.rs-online.com/webdocs/002d/0900766b8002dc8a.pdf" H 8500 4450 50  0001 C CNN
 F 4 "0.71" H 8500 4450 50  0001 C CNN "Cost"

Commit message: I put in a 4 terminal block for arming switch
Parts:
- SW1: footprint (none) -> flight-computer:TerminalBlock_TE_282834-4_1x04_P2.54mm_Horizontal
Changed lines of the file:
@@
 F 0 "SW1" H 9800 2725 50  0000 C CNN
 F 1 "SW_DPST" H 9800 2634 50  0000 C CNN
-F 2 "" H 9800 2400 50  0001 C CNN
+F 2 "flight-computer:TerminalBlock_TE_282834-4_1x04_P2.54mm_Horizontal" H 9800 2400 50  0001 C CNN
 F 3 "~" H 9800 2400 50  0001 C CNN
 	1    9800 2400

Commit message: added in the footprint for the 6 terminal block
routed the RF section with the 434 antenna
Parts:
- added J? (x2): Screw_Terminal_01x06, symbol Connector:Screw_Terminal_01x06
Changed lines of the file:
@@
 $Descr A4 11693 8268
 encoding utf-8
-Sheet 7 7
+Sheet 6 7
 Title "Pyro drivers"
 Date "2019-09-09"
@@
 	1    0    0    -1
 $EndComp
+$Comp
+L Connector:Screw_Terminal_01x06 J?
+U 1 1 5D7E8132
+P 10400 3050
+F 0 "J?" H 10480 3042 50  0000 L CNN
+F 1 "Screw_Terminal_01x06" H 10480 2951 50  0000 L CNN
+F 2 "" H 10400 3050 50  0001 C CNN
+F 3 "~" H 10400 3050 50  0001 C CNN
+	1    10400 3050
+	1    0    0    -1
+$EndComp
+$Comp
+L Connector:Screw_Terminal_01x06 J?
+U 1 1 5D7E88A1
+P 10300 4150
+F 0 "J?" H 10380 4142 50  0000 L CNN
+F 1 "Screw_Terminal_01x06" H 10380 4051 50  0000 L CNN
+F 2 "" H 10300 4150 50  0001 C CNN
+F 3 "~" H 10300 4150 50  0001 C CNN
+	1    10300 4150
+	1    0    0    -1
+$EndComp

Commit message: Done extensive routing of the board.
Parts:
- removed J3, J5: Screw_Terminal_01x04, flight-computer:TerminalBlock_TE_282834-4_1x04_P2.54mm_Horizontal, symbol Connector:Screw_Terminal_01x04
- removed SW1: SW_DPST, flight-computer:TerminalBlock_TE_282834-4_1x04_P2.54mm_Horizontal, symbol Switch:SW_DPST
- J3, J5: renamed from J?; footprint (none) -> flight-computer:TerminalBlock_TE_282834-6_1x06_P2.54mm_Horizontal
Connections:
- net +3V3: now also J5.6 (Pin_6)
- net ARMED: now also J5.5 (Pin_5)
- net FET_A: now also J3.6 (Pin_6)
- net FET_B: now also J3.4 (Pin_4)
- net FET_C: now also J5.4 (Pin_4)
- net FET_D: now also J5.2 (Pin_2)
- net Vdrive: now also J3.2 (Pin_2)
- net at J3.1 (Pin_1): now also J3.3 (Pin_3), J3.5 (Pin_5), J5.1 (Pin_1), J5.3 (Pin_3)
Other:
- note added: "Goes to a Double Pole Single Throw switch\n"
- moved on the sheet: J3, J5

Commit message: only 2 or 3 connections left to route
Parts:
- removed J3, J5: Screw_Terminal_01x06, flight-computer:TerminalBlock_TE_282834-6_1x06_P2.54mm_Horizontal, symbol Connector:Screw_Terminal_01x06
- added J3, J5: Screw_Terminal_01x04, flight-computer:TerminalBlock_TE_282834-4_1x04_P2.54mm_Horizontal, symbol Connector:Screw_Terminal_01x04
Connections:
- net FET_A: now also J3.4 (Pin_4)
- net FET_B: now also J3.2 (Pin_2)
- net FET_C: now also J5.4 (Pin_4)
- net FET_D: now also J5.2 (Pin_2)
- net Vdrive: now also J3.1 (Pin_1), J3.3 (Pin_3), J5.1 (Pin_1), J5.3 (Pin_3)
Changed lines of the file:
@@
 $Descr A4 11693 8268
 encoding utf-8
-Sheet 6 7
+Sheet 7 7
 Title "Pyro drivers"
 Date "2019-09-09"
@@
 Text Label 10000 4300 2    50   ~ 0
 FET_C
-Wire Wire Line
-	10050 4200 9750 4200
 Text Label 10050 3050 2    50   ~ 0
 FET_A
 Wire Wire Line
 	10050 3250 9750 3250
-$Comp
-L Connector:Screw_Terminal_01x06 J5
-U 1 1 5D7E88A1
-P 9550 4400
-F 0 "J5" H 9468 3875 50  0000 C CNN
-F 1 "Screw_Terminal_01x06" H 9468 3966 50  0000 C CNN
-F 2 "flight-computer:TerminalBlock_TE_282834-6_1x06_P2.54mm_Horizontal" H 9550 4400 50  0001 C CNN
-F 3 "~" H 9550 4400 50  0001 C CNN
-	1    9550 4400
-	-1   0    0    1
-$EndComp
-$Comp
-L Connector:Screw_Terminal_01x06 J3
-U 1 1 5D7E8132
-P 9550 3350
-F 0 "J3" H 9468 2825 50  0000 C CNN
-F 1 "Screw_Terminal_01x06" H 9468 2916 50  0000 C CNN
-F 2 "flight-computer:TerminalBlock_TE_282834-6_1x06_P2.54mm_Horizontal" H 9550 3350 50  0001 C CNN
-F 3 "~" H 9550 3350 50  0001 C CNN
-	1    9550 3350
-	-1   0    0    1
-$EndComp
 Text Notes 8850 2350 0    50   ~ 0
 Goes to a Double Pole Single Throw switch\n
-Wire Wire Line
-	10200 4100 10200 3950
-$Comp
-L power:+3.3V #PWR0121
-U 1 1 5D89E3F1
-P 10200 3950
-F 0 "#PWR0121" H 10200 3800 50  0001 C CNN
-F 1 "+3.3V" H 10215 4123 50  0000 C CNN
-F 2 "" H 10200 3950 50  0001 C CNN
-F 3 "" H 10200 3950 50  0001 C CNN
-	1    10200 3950
-	1    0    0    -1
-$EndComp
 Wire Wire Line
 	9750 3150 10450 3150
@@
 Wire Wire Line
 	9750 3050 10050 3050
-Wire Wire Line
-	9750 4100 10200 4100
-Wire Wire Line
-	10450 3550 10450 4400
 Connection ~ 10450 4400
 Wire Wire Line
-	10450 3350 10450 3550
-Wire Wire Line
-	9750 3550 10450 3550
-Connection ~ 10450 3550
-Wire Wire Line
 	10450 4600 10450 4400
 Wire Wire Line
 	9750 4400 10450 4400
-Text HLabel 10050 4200 2    50   Input ~ 0
-ARMED
 Wire Wire Line
 	9750 4600 10450 4600
@@
 	9750 3350 10450 3350
 Wire Wire Line
-	10750 3450 10750 3300
-Wire Wire Line
-	9750 3450 10750 3450
+	10450 3150 10450 3000
 $Comp
 L power:Vdrive #PWR0112
 U 1 1 5D7E2F36
-P 10750 3300
-F 0 "#PWR0112" H 10550 3150 50  0001 C CNN
-F 1 "Vdrive" H 10767 3473 50  0000 C CNN
-F 2 "" H 10750 3300 50  0001 C CNN
-F 3 "" H 10750 3300 50  0001 C CNN
-	1    10750 3300
+P 10450 3000
+F 0 "#PWR0112" H 10250 2850 50  0001 C CNN
+F 1 "Vdrive" H 10467 3173 50  0000 C CNN
+F 2 "" H 10450 3000 50  0001 C CNN
+F 3 "" H 10450 3000 50  0001 C CNN
+	1    10450 3000
 	1    0    0    -1
 $EndComp
@@
 Text HLabel 3700 1800 0    50   Output ~ 0
 FIRE_A
+Wire Wire Line
+	10450 3350 10450 4400
+Connection ~ 10450 3150
+$Comp
+L Connector:Screw_Terminal_01x04 J3
+U 1 1 5D9DD6B6
+P 9550 3250
+F 0 "J3" H 9468 2825 50  0000 C CNN
+F 1 "Screw_Terminal_01x04" H 9468 2916 50  0000 C CNN
+F 2 "flight-computer:TerminalBlock_TE_282834-4_1x04_P2.54mm_Horizontal" H 9550 3250 50  0001 C CNN
+F 3 "~" H 9550 3250 50  0001 C CNN
+	1    9550 3250
+	-1   0    0    1
+$EndComp
+$Comp
+L Connector:Screw_Terminal_01x04 J5
+U 1 1 5D9DEEE7
+P 9550 4500
+F 0 "J5" H 9468 4075 50  0000 C CNN
+F 1 "Screw_Terminal_01x04" H 9468 4166 50  0000 C CNN
+F 2 "flight-computer:TerminalBlock_TE_282834-4_1x04_P2.54mm_Horizontal" H 9550 4500 50  0001 C CNN
+F 3 "~" H 9550 4500 50  0001 C CNN
+	1    9550 4500
+	-1   0    0    1
+$EndComp
 $EndSCHEMATC

Commit message: added links for purchasing some of the parts
Parts:
- J3, J5: Purchase link (none) -> https://www.mouser.co.uk/ProductDetail/TE-Connectivity/2828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
Changed lines of the file:
@@
 F 2 "flight-computer:TerminalBlock_TE_282834-4_1x04_P2.54mm_Horizontal" H 9550 3250 50  0001 C CNN
 F 3 "~" H 9550 3250 50  0001 C CNN
+F 4 "https://www.mouser.co.uk/ProductDetail/TE-Connectivity/282834-4?qs=A%252Bip%252BNCYi6Pqom9P%2FaHyRQ==" H 9550 3250 50  0001 C CNN "Purchase link"
 	1    9550 3250
 	-1   0    0    1
@@
 F 2 "flight-computer:TerminalBlock_TE_282834-4_1x04_P2.54mm_Horizontal" H 9550 4500 50  0001 C CNN
 F 3 "~" H 9550 4500 50  0001 C CNN
+F 4 "https://www.mouser.co.uk/ProductDetail/TE-Connectivity/282834-4?qs=A%252Bip%252BNCYi6Pqom9P%2FaHyRQ==" H 9550 4500 50  0001 C CNN "Purchase link"
 	1    9550 4500
 	-1   0    0    1

Commit message: updated links to purchasing several components
Parts:
- U5, U6: Cost (none) -> 0.729
Changed lines of the file:
@@
 F 3 "https://www.vishay.com/docs/68986/si7232dn.pdf" H 5850 5250 50  0001 C CNN
 F 4 "https://www.mouser.co.uk/ProductDetail/Vishay-Siliconix/SI7232DN-T1-GE3?qs=%252BPu8jn5UVnH5FJ8Jo4EbFw%3D%3D" H 5850 5250 50  0001 C CNN "Purchase link"
+F 5 "0.729" H 5850 5250 50  0001 C CNN "Cost"
 	2    5850 5250
 	1    0    0    -1
@@
 F 3 "https://www.vishay.com/docs/68986/si7232dn.pdf" H 5850 4000 50  0001 C CNN
 F 4 "https://www.mouser.co.uk/ProductDetail/Vishay-Siliconix/SI7232DN-T1-GE3?qs=%252BPu8jn5UVnH5FJ8Jo4EbFw%3D%3D" H 5850 4000 50  0001 C CNN "Purchase link"
+F 5 "0.729" H 5850 4000 50  0001 C CNN "Cost"
 	1    5850 4000
 	1    0    0    -1
@@
 F 3 "https://www.vishay.com/docs/68986/si7232dn.pdf" H 5850 2600 50  0001 C CNN
 F 4 "https://www.mouser.co.uk/ProductDetail/Vishay-Siliconix/SI7232DN-T1-GE3?qs=%252BPu8jn5UVnH5FJ8Jo4EbFw%3D%3D" H 5850 2600 50  0001 C CNN "Purchase link"
+F 5 "0.729" H 5850 2600 50  0001 C CNN "Cost"
 	2    5850 2600
 	1    0    0    -1
@@
 F 3 "https://www.vishay.com/docs/68986/si7232dn.pdf" H 5850 1350 50  0001 C CNN
 F 4 "https://www.mouser.co.uk/ProductDetail/Vishay-Siliconix/SI7232DN-T1-GE3?qs=%252BPu8jn5UVnH5FJ8Jo4EbFw%3D%3D" H 5850 1350 50  0001 C CNN "Purchase link"
+F 5 "0.729" H 5850 1350 50  0001 C CNN "Cost"
 	1    5850 1350
 	1    0    0    -1
