File: Flight computer/Hardware/circuit board design v1.1/MCU.sch (KiCad schematic (older format))
At the start: 30 parts, among them J1 Conn_01x05, U11 W25Q64JVSSIM, U7 ATSAMD21J18A-AU, Y3 16MHz

Commit message: put in new acclerometers and 9dof sensor. Changed supplier from mouser to farnell and RS
Parts:
- BZ1: min_quantity (none) -> 1
- U11, Y3: min_quantity (none) -> 10
Connections:
- net MCU_PA06: no longer names the net of U7.15 (PA06)
- net MCU_PA07: no longer names the net of U7.16 (PA07)
- net MCU_PA08: no longer names the net of U7.17 (PA08)
- net MCU_PA09: no longer names the net of U7.18 (PA09)
- no-connect marks 12 -> 16
Changed lines of the file:
@@
 $Descr A4 11693 8268
 encoding utf-8
-Sheet 6 7
+Sheet 7 7
 Title ""
 Date "2019-09-09"
@@
 	8100 2600 8100 2750
 Wire Wire Line
-	5100 3500 4550 3500
-Wire Wire Line
-	5100 3600 4550 3600
-Text HLabel 4550 3500 0    50   BiDi ~ 0
-MCU_PA06
-Text HLabel 4550 3600 0    50   BiDi ~ 0
-MCU_PA07
-Wire Wire Line
-	5100 3800 4550 3800
-Wire Wire Line
 	7100 3500 7650 3500
 Wire Wire Line
@@
 F 4 "1.05" H 10600 3600 50  0001 C CNN "Cost"
 F 5 "https://uk.rs-online.com/web/p/magnetic-buzzer-components/6173081/?searchTerm=6173081&relevancy-data=636F3D3126696E3D4931384E525353746F636B4E756D6265724D504E266C753D656E266D6D3D6D61746368616C6C26706D3D5E5C647B367D247C5E5C647B377D247C5E5C647B31307D2426706F3D313426736E3D592673743D52535F53544F434B5F4E554D4245522677633D4E4F4E45267573743D3631373330383126" H 10600 3600 50  0001 C CNN "Purchase link"
+F 6 "1" H 10600 3600 50  0001 C CNN "min_quantity"
 	1    10600 3600
 	1    0    0    -1
@@
 Wire Wire Line
 	4550 2900 5100 2900
-Wire Wire Line
-	5100 3700 4550 3700
-Text HLabel 4550 3700 0    50   BiDi ~ 0
-MCU_PA08
-Text HLabel 4550 3800 0    50   BiDi ~ 0
-MCU_PA09
 Text HLabel 4550 3900 0    50   BiDi ~ 0
 MCU_PA10
@@
 F 4 "0.651" H 3300 4400 50  0001 C CNN "Cost"
 F 5 "https://uk.rs-online.com/web/p/crystal-units/1442292/" H 3300 4400 50  0001 C CNN "Purchase link"
+F 6 "10" H 3300 4400 50  0001 C CNN "min_quantity"
 	1    3300 4400
 	1    0    0    -1
@@
 F 4 "https://uk.rs-online.com/web/p/flash-memory/1882666/" H 8300 2650 50  0001 C CNN "Purchase link"
 F 5 "0.718" H 8300 2650 50  0001 C CNN "Cost"
+F 6 "10" H 8300 2650 50  0001 C CNN "min_quantity"
 	1    8300 2650
 	1    0    0    -1
@@
 	1    0    0    -1
 $EndComp
+NoConn ~ 5100 3800
+NoConn ~ 5100 3700
+NoConn ~ 5100 3600
+NoConn ~ 5100 3500
 $EndSCHEMATC
