File: Flight computer/Hardware/circuit board design v1.1/MCU.sch (KiCad schematic (older format))
At the start: 31 parts, among them J1 Conn_01x05, J5 Conn_01x04, U11 W25Q64JVSSIM, U7 ATSAMD21J18A-AU, Y3 16MHz

Commit message: put in the last bom purchase links
Parts:
- D1: Cost (none) -> 0.038; Purchase link (none) -> https://uk.rs-online.com/web/p/leds/0450711/; min_quantity (none) -> 50
- R1, R12, R25, R26: value 1.6K -> 1K; Cost 0.002 -> 0.035; Purchase link https://uk.rs-online.com/web/p/surface-mount-fixed-resistors/6789917/ -> https://uk.rs-online.com/web/p/surface-mount-fixed-resistors/2132266/
Changed lines of the file:
@@
 P 4450 6600
 F 0 "R12" H 4520 6646 50  0000 L CNN
-F 1 "1.6K" H 4520 6555 50  0000 L CNN
+F 1 "1K" H 4520 6555 50  0000 L CNN
 F 2 "Resistor_SMD:R_0603_1608Metric" V 4380 6600 50  0001 C CNN
 F 3 "~" H 4450 6600 50  0001 C CNN
-F 4 "0.002" H 4450 6600 50  0001 C CNN "Cost"
-F 5 "https://uk.rs-online.com/web/p/surface-mount-fixed-resistors/6789917/" H 4450 6600 50  0001 C CNN "Purchase link"
+F 4 "0.035" H 4450 6600 50  0001 C CNN "Cost"
+F 5 "https://uk.rs-online.com/web/p/surface-mount-fixed-resistors/2132266/" H 4450 6600 50  0001 C CNN "Purchase link"
 F 6 "50" H 4450 6600 50  0001 C CNN "min_quantity"
 	1    4450 6600
@@
 P 10200 4900
 F 0 "R25" V 10100 5000 50  0000 C CNN
-F 1 "1.6K" V 10100 4850 50  0000 C CNN
+F 1 "1K" V 10100 4850 50  0000 C CNN
 F 2 "Resistor_SMD:R_0603_1608Metric" V 10130 4900 50  0001 C CNN
 F 3 "~" H 10200 4900 50  0001 C CNN
-F 4 "0.002" H 10200 4900 50  0001 C CNN "Cost"
-F 5 "https://uk.rs-online.com/web/p/surface-mount-fixed-resistors/6789917/" H 10200 4900 50  0001 C CNN "Purchase link"
+F 4 "0.035" H 10200 4900 50  0001 C CNN "Cost"
+F 5 "https://uk.rs-online.com/web/p/surface-mount-fixed-resistors/2132266/" H 10200 4900 50  0001 C CNN "Purchase link"
 F 6 "50" H 10200 4900 50  0001 C CNN "min_quantity"
 	1    10200 4900
@@
 F 2 "LED_SMD:LED_0603_1608Metric" H 10600 4900 50  0001 C CNN
 F 3 "~" H 10600 4900 50  0001 C CNN
+F 4 "0.038" H 10600 4900 50  0001 C CNN "Cost"
+F 5 "https://uk.rs-online.com/web/p/leds/0450711/" H 10600 4900 50  0001 C CNN "Purchase link"
+F 6 "50" H 10600 4900 50  0001 C CNN "min_quantity"
 	1    10600 4900
 	-1   0    0    1
@@
 P 10200 5300
 F 0 "R26" V 10100 5400 50  0000 C CNN
-F 1 "1.6K" V 10100 5250 50  0000 C CNN
+F 1 "1K" V 10100 5250 50  0000 C CNN
 F 2 "Resistor_SMD:R_0603_1608Metric" V 10130 5300 50  0001 C CNN
 F 3 "~" H 10200 5300 50  0001 C CNN
-F 4 "0.002" H 10200 5300 50  0001 C CNN "Cost"
-F 5 "https://uk.rs-online.com/web/p/surface-mount-fixed-resistors/6789917/" H 10200 5300 50  0001 C CNN "Purchase link"
+F 4 "0.035" H 10200 5300 50  0001 C CNN "Cost"
+F 5 "https://uk.rs-online.com/web/p/surface-mount-fixed-resistors/2132266/" H 10200 5300 50  0001 C CNN "Purchase link"
 F 6 "50" H 10200 5300 50  0001 C CNN "min_quantity"
 	1    10200 5300
@@
 P 2000 4050
 F 0 "R1" H 2070 4096 50  0000 L CNN
-F 1 "1.6K" H 2070 4005 50  0000 L CNN
+F 1 "1K" H 2070 4005 50  0000 L CNN
 F 2 "Resistor_SMD:R_0603_1608Metric" V 1930 4050 50  0001 C CNN
 F 3 "~" H 2000 4050 50  0001 C CNN
-F 4 "0.002" H 2000 4050 50  0001 C CNN "Cost"
-F 5 "https://uk.rs-online.com/web/p/surface-mount-fixed-resistors/6789917/" H 2000 4050 50  0001 C CNN "Purchase link"
+F 4 "0.035" H 2000 4050 50  0001 C CNN "Cost"
+F 5 "https://uk.rs-online.com/web/p/surface-mount-fixed-resistors/2132266/" H 2000 4050 50  0001 C CNN "Purchase link"
 F 6 "50" H 2000 4050 50  0001 C CNN "min_quantity"
 	1    2000 4050
