File: Flight computer/Hardware/circuit board design v1.1/_autosave-circuit board design.kicad_pcb (KiCad board)
At the start: 4 copper layers, 30.5 x 82.6 mm, 83 parts, among them J1 Conn_01x05, J2 USB_B_Micro, J3 Screw_Terminal_01x04, J4 Conn_01x02, J6 Conn_Coaxial, J7 Conn_Coaxial, U1 LSM9DS1, U11 W25Q64JVSSIM, U14 MAX40200AUK, U15 LD3985M33R_TSOT23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

Commit message: Fully routed board v1.1 with the new high g accelerometer
Parts:
- moved C88 5.39 mm to (104.5, 90.0)
- moved C86 4.71 mm to (104.5, 95.1), turned to 180 degrees
- moved C15 2.68 mm to (97.3, 96.2)
- moved C18 2.68 mm to (93.7, 92.4)
- moved C24 2.68 mm to (94.5, 90.0)
- moved C25 2.68 mm to (94.5, 94.6)
- moved C17 2.68 mm to (95.2, 92.3)
- moved U1 2.68 mm to (99.3, 92.3)
- moved R13 1.68 mm to (117.6, 95.4), turned to 270 degrees
- moved J4 1.52 mm to (110.6, 89.5)
- moved R5 1.02 mm to (115.4, 83.2)
- moved R6 1.02 mm to (115.4, 84.7)
- moved R3 0.65 mm to (119.1, 95.4), turned to 270 degrees
- moved Y3 0.54 mm to (104.5, 92.6), turned to 90 degrees
Routing:
- net GND: track 79.7 -> 172.5 mm, vias 23 -> 53
- net /MCU/MCU_NSEL1: track 0.00 -> 37.6 mm, vias 0 -> 2
- net Net-(C35-Pad1): track 1.42 -> 38.2 mm, vias 0 -> 2
- net /MCU/MCU_PB10: track 0.00 -> 32.2 mm, vias 0 -> 2
- net /MCU/MCU_PB08: track 3.16 -> 30.9 mm, vias 1 -> 2
- net /MCU/MCU_SCLK1: track 2.63 -> 27.6 mm, vias 1 -> 2
- net /MCU/MCU_MOSI1: track 4.15 -> 28.4 mm, vias 1 -> 2
- net /MCU/MCU_PA04: track 0.00 -> 24.2 mm, vias 0 -> 2
- net /MCU/MCU_PA05: track 2.39 -> 24.9 mm, vias 0 -> 2
- net +3V3: track 161.5 -> 180.3 mm, vias 16 -> 25
- net /pyro_driver/FIRE_B: track 12.5 -> 29.5 mm, vias 0 -> 2
- net Vdrive: track 22.2 -> 38.2 mm, vias 1 -> 0
- net /MCU/MCU_MISO1: track 24.0 -> 32.2 mm
- net /MCU/MCU_PA12: track 25.6 -> 33.6 mm, vias 2 -> 0
- net /MCU/MCU_PA13: track 27.3 -> 34.4 mm, vias 2 -> 0
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- removed copper zone on B.Cu, net GND
- removed copper zone on F.Cu, net GND
