File: Flight computer/Hardware/circuit board design v1.1/power_supply.sch (KiCad schematic (older format))
At the start: 11 parts, among them J2 USB_B_Micro, J4 Conn_01x02, U14 MAX40200AUK, U15 LD3985M33R_TSOT23, U9 STF202-22T1G

Commit message: put in new acclerometers and 9dof sensor. Changed supplier from mouser to farnell and RS
Parts:
- D3, J2, U15: min_quantity (none) -> 5
- U14: min_quantity (none) -> 10
- U9: Cost 0.467 -> 0.5; Purchase link https://uk.rs-online.com/web/p/bus-terminators/1869924/ -> https://uk.farnell.com/on-semiconductor/stf202-22t1g/active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; min_quantity (none) -> 1
Changed lines of the file:
@@
 F 4 "0.36" H 5450 1700 50  0001 C CNN "Cost"
 F 5 "https://uk.farnell.com/diodes-inc/dfls130l-7/diode-schottky-30v-1a-powerdi123/dp/1843673?st=DFLS130L" H 5450 1700 50  0001 C CNN "Purchase link"
+F 6 "5" H 5450 1700 50  0001 C CNN "min_quantity"
 	1    5450 1700
 	-1   0    0    1
@@
 F 4 "0.472" H 7250 3600 50  0001 C CNN "Cost"
 F 5 "https://uk.rs-online.com/web/p/low-dropout-voltage-regulators/6868802/" H 7250 3600 50  0001 C CNN "Purchase link"
+F 6 "5" H 7250 3600 50  0001 C CNN "min_quantity"
 	1    7250 3600
 	1    0    0    -1
@@
 F 4 "https://uk.rs-online.com/web/p/node_under_construction/1697573/" H 5450 3600 50  0001 C CNN "Purchase link"
 F 5 "0.729" H 5450 3600 50  0001 C CNN "Cost"
+F 6 "10" H 5450 3600 50  0001 C CNN "min_quantity"
 	1    5450 3600
 	1    0    0    -1
@@
 F 4 "https://uk.rs-online.com/web/p/micro-usb-connectors/8486764/?relevancy-data=636F3D3126696E3D4931384E53656172636847656E65726963266C753D656E266D6D3D6D61746368616C6C7061727469616C26706D3D5E5B5C707B4C7D5C707B4E647D2D2C2F255C2E5D2B2426706F3D31333326736E3D592673723D2673743D4B4559574F52445F53494E474C455F414C5048415F4E554D455249432673633D592677633D4E4F4E45267573743D3130353031372D30303031267374613D3130353031372D3030303126&searchHistory=%7B%22enabled%22%3Atrue%7D" H 1900 1800 50  0001 C CNN "Purchase link"
 F 5 "0.694" H 1900 1800 50  0001 C CNN "Cost"
+F 6 "5" H 1900 1800 50  0001 C CNN "min_quantity"
 	1    1900 1800
 	1    0    0    -1
@@
 F 2 "Package_SO:TSOP-6_1.65x3.05mm_P0.95mm" H 3400 2500 50  0001 C CNN
 F 3 "https://www.onsemi.com/pub/Collateral/STF202-22T1-D.PDF" H 3350 2050 50  0001 C CNN
-F 4 "0.467" H 3450 2050 50  0001 C CNN "Cost"
-F 5 "https://uk.rs-online.com/web/p/bus-terminators/1869924/" H 3450 2050 50  0001 C CNN "Purchase link"
+F 4 "0.5" H 3450 2050 50  0001 C CNN "Cost"
+F 5 "https://uk.farnell.com/on-semiconductor/stf202-22t1g/active-analog-filter/dp/1651958?st=STF202-22T1G" H 3450 2050 50  0001 C CNN "Purchase link"
+F 6 "1" H 3450 2050 50  0001 C CNN "min_quantity"
 	1    3450 2050
 	-1   0    0    1

Commit message: wired up the news sensors
Parts:
- C34: footprint Capacitor_SMD:C_0402_1005Metric -> Capacitor_SMD:C_0603_1608Metric
Changed lines of the file:
@@
 F 0 "C34" H 7815 4046 50  0000 L CNN
 F 1 "10nF" H 7815 3955 50  0000 L CNN
-F 2 "Capacitor_SMD:C_0402_1005Metric" H 7738 3850 50  0001 C CNN
+F 2 "Capacitor_SMD:C_0603_1608Metric" H 7738 3850 50  0001 C CNN
 F 3 "~" H 7700 4000 50  0001 C CNN
 	1    7700 4000

Commit message: put in logo for V1.1
Parts:
- C34: Cost (none) -> 0.031; Purchase link (none) -> https://uk.rs-online.com/web/p/mlccs-multilayer-ceramic-cap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; min_quantity (none) -> 100
- C35, C36: Cost (none) -> 0.01; Purchase link (none) -> https://uk.rs-online.com/web/p/mlccs-multilayer-ceramic-cap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; min_quantity (none) -> 250
- R28, R29: value 100K -> 120K; Cost (none) -> 0.035; Purchase link (none) -> https://uk.rs-online.com/web/p/surface-mount-fixed-resistor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; min_quantity (none) -> 50
Changed lines of the file:
@@
 F 2 "Capacitor_SMD:C_0603_1608Metric" H 7738 3850 50  0001 C CNN
 F 3 "~" H 7700 4000 50  0001 C CNN
+F 4 "0.031" H 7700 4000 50  0001 C CNN "Cost"
+F 5 "https://uk.rs-online.com/web/p/mlccs-multilayer-ceramic-capacitors/8391727/" H 7700 4000 50  0001 C CNN "Purchase link"
+F 6 "100" H 7700 4000 50  0001 C CNN "min_quantity"
 	1    7700 4000
 	1    0    0    -1
@@
 F 2 "Capacitor_SMD:C_0603_1608Metric" H 8138 3850 50  0001 C CNN
 F 3 "~" H 8100 4000 50  0001 C CNN
+F 4 "0.01" H 8100 4000 50  0001 C CNN "Cost"
+F 5 "https://uk.rs-online.com/web/p/mlccs-multilayer-ceramic-capacitors/1358359/" H 8100 4000 50  0001 C CNN "Purchase link"
+F 6 "250" H 8100 4000 50  0001 C CNN "min_quantity"
 	1    8100 4000
 	1    0    0    -1
@@
 F 2 "Capacitor_SMD:C_0603_1608Metric" H 6688 3850 50  0001 C CNN
 F 3 "~" H 6650 4000 50  0001 C CNN
+F 4 "0.01" H 6650 4000 50  0001 C CNN "Cost"
+F 5 "https://uk.rs-online.com/web/p/mlccs-multilayer-ceramic-capacitors/1358359/" H 6650 4000 50  0001 C CNN "Purchase link"
+F 6 "250" H 6650 4000 50  0001 C CNN "min_quantity"
 	1    6650 4000
 	1    0    0    -1
@@
 P 4150 4800
 F 0 "R28" H 4220 4846 50  0000 L CNN
-F 1 "100K" H 4220 4755 50  0000 L CNN
+F 1 "120K" H 4220 4755 50  0000 L CNN
 F 2 "Resistor_SMD:R_0603_1608Metric" V 4080 4800 50  0001 C CNN
 F 3 "~" H 4150 4800 50  0001 C CNN
+F 4 "0.035" H 4150 4800 50  0001 C CNN "Cost"
+F 5 "https://uk.rs-online.com/web/p/surface-mount-fixed-resistors/6789715/" H 4150 4800 50  0001 C CNN "Purchase link"
+F 6 "50" H 4150 4800 50  0001 C CNN "min_quantity"
 	1    4150 4800
 	1    0    0    -1
@@
 P 4150 5300
 F 0 "R29" H 4220 5346 50  0000 L CNN
-F 1 "100K" H 4220 5255 50  0000 L CNN
+F 1 "120K" H 4220 5255 50  0000 L CNN
 F 2 "Resistor_SMD:R_0603_1608Metric" V 4080 5300 50  0001 C CNN
 F 3 "~" H 4150 5300 50  0001 C CNN
+F 4 "0.035" H 4150 5300 50  0001 C CNN "Cost"
+F 5 "https://uk.rs-online.com/web/p/surface-mount-fixed-resistors/6789715/" H 4150 5300 50  0001 C CNN "Purchase link"
+F 6 "50" H 4150 5300 50  0001 C CNN "min_quantity"
 	1    4150 5300
 	1    0    0    -1
