File: Flight computer/Hardware/circuit board design v1.1/GPS.sch (KiCad schematic (older format))
At the start: 7 parts, among them J6 Conn_Coaxial, U4 MAX-M8C

Commit message: put in new acclerometers and 9dof sensor. Changed supplier from mouser to farnell and RS
Parts:
- J6: Cost 0.746 -> 0.617; Purchase link https://uk.farnell.com/hirose-hrs/u-fl-r-smt-1-10/rf-coaxia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 -> https://uk.rs-online.com/web/p/coaxial-plugs-sockets/702542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
- U4: min_quantity (none) -> 1
Changed lines of the file:
@@
 F 2 "Connector_Coaxial:U.FL_Hirose_U.FL-R-SMT-1_Vertical" H 8450 4050 50  0001 C CNN
 F 3 "https://www.mouser.co.uk/datasheet/2/185/U.FL_catalog-939761.pdf" H 8450 4050 50  0001 C CNN
-F 4 "0.746" H 8450 4050 50  0001 C CNN "Cost"
-F 5 "https://uk.farnell.com/hirose-hrs/u-fl-r-smt-1-10/rf-coaxial-u-fl-straight-jack/dp/1688077?st=ufl" H 8450 4050 50  0001 C CNN "Purchase link"
+F 4 "0.617" H 8450 4050 50  0001 C CNN "Cost"
+F 5 "https://uk.rs-online.com/web/p/coaxial-plugs-sockets/7025425/" H 8450 4050 50  0001 C CNN "Purchase link"
 F 6 "10" H 8450 4050 50  0001 C CNN "min_quantity"
 	1    8450 4050
@@
 F 4 "11.99" H 6050 4050 50  0001 C CNN "Cost"
 F 5 "https://store.uputronics.com/index.php?route=product/product&product_id=71&search=ublox" H 6050 4050 50  0001 C CNN "Purchase link"
+F 6 "1" H 6050 4050 50  0001 C CNN "min_quantity"
 	1    6050 4050
 	1    0    0    -1

Commit message: put in logo for V1.1
Parts:
- C11: Cost (none) -> 0.01; Purchase link (none) -> https://uk.rs-online.com/web/p/mlccs-multilayer-ceramic-cap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; min_quantity (none) -> 50
- C12: Cost (none) -> 0.07; Purchase link (none) -> https://uk.rs-online.com/web/p/mlccs-multilayer-ceramic-cap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; min_quantity (none) -> 100
- C8: Cost (none) -> 0.031; Purchase link (none) -> https://uk.rs-online.com/web/p/mlccs-multilayer-ceramic-cap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; min_quantity (none) -> 100
- R2: Purchase link (none) -> https://uk.rs-online.com/web/p/surface-mount-fixed-resistor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; min_quantity (none) -> 50
Changed lines of the file:
@@
 F 2 "Resistor_SMD:R_0402_1005Metric" V 6880 3100 50  0001 C CNN
 F 3 "~" H 6950 3100 50  0001 C CNN
+F 4 "https://uk.rs-online.com/web/p/surface-mount-fixed-resistors/6788703/" H 6950 3100 50  0001 C CNN "Purchase link"
+F 5 "50" H 6950 3100 50  0001 C CNN "min_quantity"
 	1    6950 3100
 	0    1    1    0
@@
 F 2 "Capacitor_SMD:C_0402_1005Metric" H 8400 2750 50  0001 C CNN
 F 3 "~" H 8400 2750 50  0001 C CNN
+F 4 "0.031" H 8400 2750 50  0001 C CNN "Cost"
+F 5 "https://uk.rs-online.com/web/p/mlccs-multilayer-ceramic-capacitors/8391727/" H 8400 2750 50  0001 C CNN "Purchase link"
+F 6 "100" H 8400 2750 50  0001 C CNN "min_quantity"
 	1    8400 2750
 	1    0    0    -1
@@
 F 1 "100nF" H 5208 2805 50  0000 R CNN
 F 2 "Capacitor_SMD:C_0603_1608Metric" H 5300 2850 50  0001 C CNN
-F 3 "~" H 5300 2850 50  0001 C CNN
+F 3 "https://docs-emea.rs-online.com/webdocs/0dc2/0900766b80dc2409.pdf" H 5300 2850 50  0001 C CNN
+F 4 "0.01" H 5300 2850 50  0001 C CNN "Cost"
+F 5 "https://uk.rs-online.com/web/p/mlccs-multilayer-ceramic-capacitors/6983251/" H 5300 2850 50  0001 C CNN "Purchase link"
+F 6 "50" H 5300 2850 50  0001 C CNN "min_quantity"
 	1    5300 2850
 	1    0    0    -1
@@
 F 1 "10uF" H 5558 2805 50  0000 R CNN
 F 2 "Capacitor_SMD:C_0603_1608Metric" H 5650 2850 50  0001 C CNN
-F 3 "~" H 5650 2850 50  0001 C CNN
+F 3 "https://docs-emea.rs-online.com/webdocs/13b3/0900766b813b3e64.pdf" H 5650 2850 50  0001 C CNN
+F 4 "0.07" H 5650 2850 50  0001 C CNN "Cost"
+F 5 "https://uk.rs-online.com/web/p/mlccs-multilayer-ceramic-capacitors/8467293/" H 5650 2850 50  0001 C CNN "Purchase link"
+F 6 "100" H 5650 2850 50  0001 C CNN "min_quantity"
 	1    5650 2850
 	1    0    0    -1

Commit message: changed GPS to M8Q and included the diode from V bus to foot print which I missed out
Parts:
- removed U4: MAX-M8C, RF_GPS:ublox_MAX, symbol RF_GPS:MAX-M8C
- added U?: MAX-M8Q, RF_GPS:ublox_MAX, symbol RF_GPS:MAX-M8Q
- L2: Cost (none) -> 0.08; Purchase link (none) -> https://uk.rs-online.com/web/p/wire-wound-surface-mount-ind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; min_quantity (none) -> 10
- R2: Cost (none) -> 0.002
Connections:
- net +3V3: now also U?.6 (V_BCKP), U?.7 (VCC_IO), U?.8 (VCC)
- net GND: now also U?.1 (GND), U?.10 (GND), U?.12 (GND)
- net GPS_1PPS: now also U?.4 (TIMEPULSE)
- net GPS_NRES: now also U?.9 (~RESET)
- net GPS_NSAFEBOOT: now also U?.18 (~SAFEBOOT)
- net GPS_RXD: now also U?.3 (RXD)
- net GPS_SCL: now also U?.17 (SCL)
- net GPS_SDA: now also U?.16 (SDA)
- net GPS_TXD: now also U?.2 (TXD)
- net at J6.1 (In), L2.2: now also U?.11 (RF_IN)
- net at R2.2: now also U?.14 (VCC_RF)
Changed lines of the file:
@@
 F 2 "Resistor_SMD:R_0402_1005Metric" H 7650 3650 50  0001 C CNN
 F 3 "~" H 7650 3650 50  0001 C CNN
+F 4 "0.08" H 7650 3650 50  0001 C CNN "Cost"
+F 5 "https://uk.rs-online.com/web/p/wire-wound-surface-mount-inductors/7254923/" H 7650 3650 50  0001 C CNN "Purchase link"
+F 6 "10" H 7650 3650 50  0001 C CNN "min_quantity"
 	1    7650 3650
 	1    0    0    -1
@@
 F 4 "https://uk.rs-online.com/web/p/surface-mount-fixed-resistors/6788703/" H 6950 3100 50  0001 C CNN "Purchase link"
 F 5 "50" H 6950 3100 50  0001 C CNN "min_quantity"
+F 6 "0.002" H 6950 3100 50  0001 C CNN "Cost"
 	1    6950 3100
 	0    1    1    0
@@
 Wire Wire Line
 	5300 3050 5650 3050
+Wire Wire Line
+	6050 3350 6050 3300
+Wire Wire Line
+	6050 3300 5950 3300
+Connection ~ 5950 3300
+Wire Wire Line
+	5950 3300 5950 2650
 $Comp
-L RF_GPS:MAX-M8C U4
-U 1 1 5D610F77
+L RF_GPS:MAX-M8Q U?
+U 1 1 5D91C1E4
 P 6050 4050
-F 0 "U4" H 6050 4900 50  0000 C CNN
-F 1 "MAX-M8C" H 6500 3300 50  0000 C CNN
+F 0 "U?" H 6050 3261 50  0000 C CNN
+F 1 "MAX-M8Q" H 5600 3200 50  0000 C CNN
 F 2 "RF_GPS:ublox_MAX" H 6450 3400 50  0001 C CNN
 F 3 "https://www.u-blox.com/sites/default/files/MAX-M8-FW3_DataSheet_%28UBX-15031506%29.pdf" H 6050 4050 50  0001 C CNN
@@
 	1    0    0    -1
 $EndComp
-Wire Wire Line
-	6050 3350 6050 3300
-Wire Wire Line
-	6050 3300 5950 3300
-Connection ~ 5950 3300
-Wire Wire Line
-	5950 3300 5950 2650
 $EndSCHEMATC

Commit message: added in grove connector for break out pins. Made a new software framework for SAMD
Parts:
- gave numbers to parts that had none: 1
Changed lines of the file:
@@
 	5950 3300 5950 2650
 $Comp
-L RF_GPS:MAX-M8Q U?
+L RF_GPS:MAX-M8Q U4
 U 1 1 5D91C1E4
 P 6050 4050
-F 0 "U?" H 6050 3261 50  0000 C CNN
+F 0 "U4" H 6050 3261 50  0000 C CNN
 F 1 "MAX-M8Q" H 5600 3200 50  0000 C CNN
 F 2 "RF_GPS:ublox_MAX" H 6450 3400 50  0001 C CNN
